File: PCB_DEV_BOARD-ESP12/BHOnOfreDevBoard.sch (EAGLE design)
At the start: 22 parts, among them K1 OMRON-G3MB-202P-SSR2, K2 OMRON-G3MB-202P-SSR2, Q1 S8050, Q2 S8050

Commit message: Organização de ficheiros e versões do OnOfre, devenvolvimento da dev board
Parts:
- added J8, J9: (no value), SparkFun-Connectors:CONN_01
Connections:
- removed net GND1: J4.1, J4.2, J4.3, J4.4, J4.5, J4.6, J4.7, J4.8
- removed net N$10: R11.1, U2.GPIO15
- net GPIO15: now also R11.1, U2.GPIO15
- net R1: now also J8.1
- net R2: now also J9.1
- net VCC: now also J4.1, J4.2, J4.3, J4.4, J4.5, J4.6, J4.7, J4.8
Other:
- note added: "DEV BOARD"

Commit message: melhoramentos nas pistas da dev board
Parts:
- added SW1: B3U-1000P-2P-SMD, Seeed-Switch:SMD-BUTTON(2P-3.0X2.5X1.2+0.4MM)-B3U-1000P-2P-SMD
Connections:
- net GND: now also SW1.2
- net RESET: now also SW1.1
Changed lines of the file:
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@@
 <part name="J8" library="SparkFun-Connectors" library_urn="urn:adsk.eagle:library:513" deviceset="CONN_01" device="" package3d_urn="urn:adsk.eagle:package:38028/1"/>
 <part name="J9" library="SparkFun-Connectors" library_urn="urn:adsk.eagle:library:513" deviceset="CONN_01" device="" package3d_urn="urn:adsk.eagle:package:38028/1"/>
+<part name="SW1" library="Seeed-Switch" library_urn="urn:adsk.eagle:library:476" deviceset="SMD-BUTTON(2P-3.0X2.5X1.2+0.4MM)" device="-B3U-1000P-2P-SMD" package3d_urn="urn:adsk.eagle:package:32999/1" value="B3U-1000P-2P-SMD"/>
 </parts>
 <sheets>
@@
 <instance part="J8" gate="G$1" x="205.74" y="53.34"/>
 <instance part="J9" gate="G$1" x="205.74" y="43.18"/>
+<instance part="SW1" gate="G$1" x="58.42" y="93.98"/>
 </instances>
 <busses>
@@
 <label x="144.78" y="152.4" size="1.778" layer="95" xref="yes"/>
 </segment>
+<segment>
+<pinref part="SW1" gate="G$1" pin="2"/>
+<wire x1="66.04" y1="93.98" x2="81.28" y2="93.98" width="0.1524" layer="91"/>
+<label x="81.28" y="93.98" size="1.778" layer="95" xref="yes"/>
+</segment>
 </net>
 <net name="VCC" class="0">
@@
 <label x="134.62" y="142.24" size="1.778" layer="95" xref="yes"/>
 </segment>
-</net>
+<segment>
+<pinref part="SW1" gate="G$1" pin="1"/>
+<wire x1="50.8" y1="93.98" x2="38.1" y2="93.98" width="0.1524" layer="91"/>
+<label x="38.1" y="93.98" size="1.778" layer="95" rot="R180" xref="yes"/>
+</segment>
+</net>

Commit message: problema de pull up dos relés resolvido, alteração  da fonte de 3.3v para 5v
Parts:
- removed J2, J3, J4, J5: (no value), SparkFun-Connectors:CONN_08"
- added R2, R3: 10k, resistor:R-EU_R0603
- added SW2: B3U-1000P-2P-SMD, Seeed-Switch:SMD-BUTTON(2P-3.0X2.5X1.2+0.4MM)-B3U-1000P-2P-SMD
- added U1: (no value), SparkFun-IC-Power:V_REG_LM1117SOT223
- R1, R11, R4: value 47k -> 10k
Connections:
- new net 3V3: C4.1, J7.1, R10.2, R8.2, R9.2, U1.OUT, U2.VCC
- net GND: now also R2.1, R3.1, SW2.2, U1.ADJ; no longer J2.1, J2.2, J2.3, J2.4, J2.5, J2.6, J2.7, J2.8, J5.1, J5.2, J5.3, J5.4, J5.5, J5.6, J5.7, J5.8
- net GPIO0: now also SW2.1
- net N$13: now also R2.2
- net N$7: now also R3.2
- net NEUTRAL_ONE_OUT: now also J1.2; no longer J1.1
- net NEUTRAL_TWO_OUT: now also J1.1; no longer J1.2
- net VCC: now also U1.IN; no longer C4.1, J3.1, J3.2, J3.3, J3.4, J3.5, J3.6, J3.7, J3.8, J4.1, J4.2, J4.3, J4.4, J4.5, J4.6, J4.7, J4.8, J7.1, R10.2, R8.2, R9.2, U2.VCC
Other:
- note added: "HLK-PM05"
- note removed: "HLK-PM03"
