File: PCB_IN_DEVELOPMENT/PCB_SQUARE_BOARD-ESP12/BHOnOfreSquareBoard.brd (EAGLE design)
At the start: 47.6 x 47.7 mm, 23 parts, among them J1 4p, J6 8p, J7 8p, K1 OMRON-G3MB-202P-SSR2, K2 OMRON-G3MB-202P-SSR2, Q1 S8050, Q2 S8050, U1 LM1117, U2 esp12

Commit message: OnOfre Square rev2 80% pronto
Parts:
- moved D3 46.2 mm to (37.2, 2.57), flipped to the bottom, turned to 180 degrees
- moved R9 41.4 mm to (9.70, 43.9), turned to 180 degrees
- moved R8 26.3 mm to (20.4, 37.4)
- moved RESET 22.9 mm to (28.4, 32.5), flipped to the bottom, turned to 0 degrees
- moved U1 22.1 mm to (7.20, 27.8), turned to 180 degrees
- moved FLASH 19.5 mm to (28.4, 27.4), flipped to the bottom, turned to 0 degrees
- moved R10 17.7 mm to (29.3, 36.1), flipped to the bottom, turned to 0 degrees
- moved R11 16.3 mm to (10.3, 35.0), turned to 180 degrees
- moved C4 13.9 mm to (8.15, 37.5), turned to 0 degrees
- moved F1 13.5 mm to (28.5, 2.03), turned to 0 degrees
- moved K1 10.7 mm to (37.3, 8.03), turned to 0 degrees
- moved Q1 9.09 mm to (42.6, 4.09), turned to 270 degrees
- moved U2 8.58 mm to (33.3, 31.4)
- moved R3 8.51 mm to (39.0, 3.90), turned to 90 degrees
- moved J7 8.44 mm to (25.1, 43.0)
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Routing:
- net GND: track 0.23 -> 86.1 mm
- net VCC: track 0.00 -> 69.3 mm
- net 3V3: track 0.76 -> 51.3 mm
- net CH_PD: track 0.00 -> 34.8 mm
- net GPIO0: track 0.00 -> 32.5 mm
- net GPIO15: track 0.00 -> 25.6 mm
- net RESET: track 0.00 -> 24.5 mm
- net GPIO05: track 1.48 -> 17.2 mm
- net N$2: track 0.00 -> 12.4 mm
- net NEUTRAL_IN_FUSED: track 0.00 -> 11.7 mm
- net ADC: track 0.00 -> 6.14 mm
- net GPIO16: track 0.00 -> 5.26 mm
- net TX: track 0.00 -> 5.09 mm
- net N$7: track 0.00 -> 5.07 mm
- net GPIO04: track 0.00 -> 4.47 mm
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Other:
- board text added: "OnOfre rev2"
- board text removed: "OnOfre rev1"
