File: PCB_NOT_TESTED/PCB_SQUARE_BOARD-ESP12/BHOnOfreSquareBoard.sch (EAGLE design)
At the start: 23 parts, among them J1 4p, J6 8p, J7 8p, K1 OMRON-G3MB-202P-SSR2, K2 OMRON-G3MB-202P-SSR2, Q1 S8050, Q2 S8050, U1 LM1117, U2 esp12

Commit message: Square Rev2 pronto para testes
Parts:
- removed J1: 4p, SparkFun-Connectors:CONN_04SCREW
- added X2: PLUG, con-wago-500:W237-4
- C4: value 100nF -> 100nf; device SparkFun-Capacitors:10NF-0603-50V-10% -> Seeed-Capacitor:CERAMIC-100NF-50V-10%-X7R(0805)
- U$2: value HLK-PM03 -> HKLPM01; device PowerSocket:HLK-PM03 -> HKLPM01:HKLPM01
- renumbered Q2 to JY3, U1 to AMS1117
Connections:
- removed net FASE: J1.3, U$2.AC2
- new net FASE_IN: U$2.AC2, X2-2.KL
- net NEUTRAL_IN: now also X2-1.KL; no longer J1.4
- net NEUTRAL_ONE_OUT: now also X2-3.KL; no longer J1.2
- net NEUTRAL_TWO_OUT: now also X2-4.KL; no longer J1.1
