File: PCB/OnOnfre_dual_rev2/OnOnfre_dual_rev2.sch (EAGLE design)
At the start: 28 parts, among them J6 8p, J7 8p, K1 OMRON-G3MB-202P-SSR2, K2 OMRON-G3MB-202P-SSR2, Q1 S8050, U2 esp12, X2 PLUG

Commit message: Organização do repositorio
Parts:
- removed C1: 0.1uf, Seeed-Capacitor:CERAMIC-100NF-50V-10%-X7R(0805)
- removed C2: 1nf, Seeed-Capacitor:CERAMIC-100NF-50V-10%-X7R(0805)
- removed R5: 10k, resistor:R-EU_R0603
- removed R6: 39k, resistor:R-EU_R0603
- removed U$1: ACS712, SparkFun-Sensors:ACS712
Connections:
- removed net N$4: C2.1, U$1.FILT
- removed net NEUTRAL_IN_FUSED_OUT: K1.DS2, K2.DS2, U$1.IP+@1, U$1.IP+@2
- removed net SOUT: R6.1, U$1.VOUT
- net ADC: no longer R5.1, R6.2
- net GND: no longer C1.2, C2.2, R5.2, U$1.GND
- net NEUTRAL_IN_FUSED: now also K1.DS2, K2.DS2; no longer U$1.IP-@3, U$1.IP-@4
- net VCC: no longer C1.1, U$1.VCC
Other:
- note added: "REV1"
- note removed: "REV3"
Changed lines of the file:
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@@
 <?xml version="1.0" encoding="utf-8"?>
 <!DOCTYPE eagle SYSTEM "eagle.dtd">
-<eagle version="8.5.2">
+<eagle version="8.6.0">
 <drawing>
 <settings>
@@
 <part name="FLASH" library="Seeed-Switch" library_urn="urn:adsk.eagle:library:476" deviceset="SMD-BUTTON(2P-3.0X2.5X1.2+0.4MM)" device="-B3U-1000P-2P-SMD" package3d_urn="urn:adsk.eagle:package:32999/1" value="B3U-1000P-2P-SMD"/>
 <part name="X2" library="con-wago-500" library_urn="urn:adsk.eagle:library:195" deviceset="W237-4" device="" package3d_urn="urn:adsk.eagle:package:10695/1" value="PLUG"/>
-<part name="U$1" library="SparkFun-Sensors" library_urn="urn:adsk.eagle:library:534" deviceset="ACS712" device="" package3d_urn="urn:adsk.eagle:package:39975/1" value="ACS712"/>
-<part name="C1" library="Seeed-Capacitor" library_urn="urn:adsk.eagle:library:464" deviceset="CERAMIC-100NF-50V-10%-X7R(0805)" device="" package3d_urn="urn:adsk.eagle:package:32459/1" value="0.1uf"/>
-<part name="C2" library="Seeed-Capacitor" library_urn="urn:adsk.eagle:library:464" deviceset="CERAMIC-100NF-50V-10%-X7R(0805)" device="" package3d_urn="urn:adsk.eagle:package:32459/1" value="1nf"/>
-<part name="R5" library="resistor" library_urn="urn:adsk.eagle:library:348" deviceset="R-EU_" device="R0603" package3d_urn="urn:adsk.eagle:package:26057/1" value="10k"/>
-<part name="R6" library="resistor" library_urn="urn:adsk.eagle:library:348" deviceset="R-EU_" device="R0603" package3d_urn="urn:adsk.eagle:package:26057/1" value="39k"/>
 </parts>
 <sheets>
@@
 <text x="175.26" y="167.64" size="6.4516" layer="95">BH ON OFRE 12</text>
 <text x="53.34" y="157.48" size="5.08" layer="95">ESP8266-12</text>
-<text x="175.26" y="160.02" size="6.4516" layer="95">REV3</text>
+<text x="175.26" y="160.02" size="6.4516" layer="95">REV1</text>
 </plain>
 <instances>
@@
 <instance part="X2" gate="-3" x="2.54" y="15.24"/>
 <instance part="X2" gate="-4" x="2.54" y="10.16"/>
-<instance part="U$1" gate="G$1" x="218.44" y="66.04"/>
-<instance part="C1" gate="G$1" x="248.92" y="66.04" rot="R270"/>
-<instance part="C2" gate="G$1" x="243.84" y="58.42" rot="R270"/>
-<instance part="R5" gate="G$1" x="223.52" y="83.82" rot="R180"/>
-<instance part="R6" gate="G$1" x="248.92" y="83.82" rot="R180"/>
 </instances>
 <busses>
@@
 <label x="88.9" y="109.22" size="1.778" layer="95" xref="yes"/>
 </segment>
-<segment>
-<wire x1="248.92" y1="63.5" x2="248.92" y2="62.23" width="0.1524" layer="91"/>
-<wire x1="248.92" y1="62.23" x2="248.92" y2="58.42" width="0.1524" layer="91"/>
-<wire x1="248.92" y1="58.42" x2="254" y2="58.42" width="0.1524" layer="91"/>
-<label x="254" y="58.42" size="1.778" layer="95" xref="yes"/>
-<pinref part="C1" gate="G$1" pin="2"/>
-<junction x="248.92" y="62.23"/>
-</segment>
-<segment>
-<pinref part="U$1" gate="G$1" pin="GND"/>
-<wire x1="231.14" y1="63.5" x2="238.76" y2="63.5" width="0.1524" layer="91"/>
-<wire x1="238.76" y1="63.5" x2="238.76" y2="53.34" width="0.1524" layer="91"/>
-<wire x1="238.76" y1="53.34" x2="243.84" y2="53.34" width="0.1524" layer="91"/>
-<wire x1="243.84" y1="53.34" x2="243.84" y2="54.61" width="0.1524" layer="91"/>
-<pinref part="C2" gate="G$1" pin="2"/>
-<wire x1="243.84" y1="54.61" x2="243.84" y2="55.88" width="0.1524" layer="91"/>
-<junction x="243.84" y="54.61"/>
-<label x="243.84" y="53.34" size="1.778" layer="95" xref="yes"/>
-</segment>
-<segment>
-<pinref part="R5" gate="G$1" pin="2"/>
-<wire x1="218.44" y1="83.82" x2="208.28" y2="83.82" width="0.1524" layer="91"/>
-<label x="208.28" y="83.82" size="1.778" layer="95" rot="R180" xref="yes"/>
-</segment>
 </net>
 <net name="VCC" class="0">
@@
 </segment>
 <segment>
-<label x="144.78" y="66.04" size="1.778" layer="95" xref="yes"/>
+<label x="149.86" y="66.04" size="1.778" layer="95" xref="yes"/>
 <pinref part="D3" gate="G$1" pin="+"/>
-<wire x1="143.51" y1="66.04" x2="144.78" y2="66.04" width="0.1524" layer="91"/>
+<wire x1="143.51" y1="66.04" x2="149.86" y2="66.04" width="0.1524" layer="91"/>
 </segment>
 <segment>
@@
 <wire x1="160.02" y1="111.76" x2="147.32" y2="111.76" width="0.1524" layer="91"/>
 <label x="147.32" y="111.76" size="1.778" layer="95" rot="R180" xref="yes"/>
-</segment>
-<segment>
-<pinref part="U$1" gate="G$1" pin="VCC"/>
-<wire x1="231.14" y1="71.12" x2="248.92" y2="71.12" width="0.1524" layer="91"/>
-<label x="254" y="71.12" size="1.778" layer="95" xref="yes"/>
-<wire x1="248.92" y1="71.12" x2="254" y2="71.12" width="0.1524" layer="91"/>
-<wire x1="248.92" y1="68.58" x2="248.92" y2="69.85" width="0.1524" layer="91"/>
-<pinref part="C1" gate="G$1" pin="1"/>
-<wire x1="248.92" y1="69.85" x2="248.92" y2="71.12" width="0.1524" layer="91"/>
-<junction x="248.92" y="69.85"/>
 </segment>
 </net>
@@
 </segment>
 <segment>
-<pinref part="U$1" gate="G$1" pin="IP-@4"/>
-<wire x1="203.2" y1="63.5" x2="190.5" y2="63.5" width="0.1524" layer="91"/>
-<wire x1="190.5" y1="63.5" x2="190.5" y2="66.04" width="0.1524" layer="91"/>
-<wire x1="190.5" y1="66.04" x2="203.2" y2="66.04" width="0.1524" layer="91"/>
-<wire x1="203.2" y1="66.04" x2="205.74" y2="66.04" width="0.1524" layer="91"/>
-<wire x1="190.5" y1="63.5" x2="185.42" y2="63.5" width="0.1524" layer="91"/>
-<label x="185.42" y="63.5" size="1.778" layer="95" rot="R180" xref="yes"/>
-<pinref part="U$1" gate="G$1" pin="IP-@3"/>
-<junction x="203.2" y="66.04"/>
-<junction x="190.5" y="63.5"/>
+<pinref part="K2" gate="G$1" pin="DS2"/>
+<wire x1="58.42" y1="43.18" x2="35.56" y2="43.18" width="0.1524" layer="91"/>
+<label x="35.56" y="43.18" size="1.778" layer="95" rot="R180" xref="yes"/>
+</segment>
+<segment>
+<pinref part="K1" gate="G$1" pin="DS2"/>
+<wire x1="58.42" y1="71.12" x2="35.56" y2="71.12" width="0.1524" layer="91"/>
+<label x="35.56" y="71.12" size="1.778" layer="95" rot="R180" xref="yes"/>
 </segment>
 </net>
@@
 <wire x1="129.54" y1="139.7" x2="147.32" y2="139.7" width="0.1524" layer="91"/>
 <label x="147.32" y="139.7" size="1.778" layer="95" xref="yes"/>
-</segment>
-<segment>
-<pinref part="R5" gate="G$1" pin="1"/>
-<wire x1="228.6" y1="83.82" x2="236.22" y2="83.82" width="0.1524" layer="91"/>
-<pinref part="R6" gate="G$1" pin="2"/>
-<wire x1="236.22" y1="83.82" x2="243.84" y2="83.82" width="0.1524" layer="91"/>
-<wire x1="236.22" y1="83.82" x2="236.22" y2="93.98" width="0.1524" layer="91"/>
-<label x="236.22" y="93.98" size="1.778" layer="95" xref="yes"/>
 </segment>
 </net>
@@
 </segment>
 </net>
-<net name="N$4" class="0">
-<segment>
-<pinref part="U$1" gate="G$1" pin="FILT"/>
-<wire x1="231.14" y1="66.04" x2="243.84" y2="66.04" width="0.1524" layer="91"/>
-<wire x1="243.84" y1="60.96" x2="243.84" y2="62.23" width="0.1524" layer="91"/>
-<pinref part="C2" gate="G$1" pin="1"/>
-<wire x1="243.84" y1="62.23" x2="243.84" y2="66.04" width="0.1524" layer="91"/>
-<junction x="243.84" y="62.23"/>
-</segment>
-</net>
-<net name="NEUTRAL_IN_FUSED_OUT" class="0">
-<segment>
-<pinref part="U$1" gate="G$1" pin="IP+@2"/>
-<wire x1="203.2" y1="68.58" x2="190.5" y2="68.58" width="0.1524" layer="91"/>
-<pinref part="U$1" gate="G$1" pin="IP+@1"/>
-<wire x1="190.5" y1="71.12" x2="203.2" y2="71.12" width="0.1524" layer="91"/>
-<wire x1="190.5" y1="68.58" x2="190.5" y2="71.12" width="0.1524" layer="91"/>
-<label x="190.5" y="71.12" size="1.778" layer="95" rot="R180" xref="yes"/>
-</segment>
-<segment>
-<pinref part="K2" gate="G$1" pin="DS2"/>
-<wire x1="58.42" y1="43.18" x2="30.48" y2="43.18" width="0.1524" layer="91"/>
-<label x="30.48" y="43.18" size="1.778" layer="95" rot="R180" xref="yes"/>
-</segment>
-<segment>
-<pinref part="K1" gate="G$1" pin="DS2"/>
-<wire x1="58.42" y1="71.12" x2="27.94" y2="71.12" width="0.1524" layer="91"/>
-<label x="27.94" y="71.12" size="1.778" layer="95" rot="R180" xref="yes"/>
-</segment>
-</net>
-<net name="SOUT" class="0">
-<segment>
-<pinref part="U$1" gate="G$1" pin="VOUT"/>
-<wire x1="231.14" y1="68.58" x2="236.22" y2="68.58" width="0.1524" layer="91"/>
-<label x="236.22" y="68.58" size="1.778" layer="95" xref="yes"/>
-</segment>
-<segment>
-<pinref part="R6" gate="G$1" pin="1"/>
-<wire x1="254" y1="83.82" x2="259.08" y2="83.82" width="0.1524" layer="91"/>
-<label x="259.08" y="83.82" size="1.778" layer="95" rot="R90" xref="yes"/>
-</segment>
-</net>
