File: PCB/OnOnfre_dual_rev3.1/OnOfre_2ADSP.sch (EAGLE design)
At the start: 23 parts, among them J1 4p, J6 8p, J7 8p, K1 OMRON-G3MB-202P-SSR2, K2 OMRON-G3MB-202P-SSR2, Q1 S8050, Q2 S8050, U1 LM1117, U2 esp12

Commit message: Rev3.1 dual
Parts:
- removed J1: 4p, SparkFun-Connectors:CONN_04SCREW
- added R5: VARISTORS07K230, varistor:VARISTORS07K230
- added X1: (no value), con-wago-500:W237-4
- C4: value 100nF -> 100NF; device SparkFun-Capacitors:10NF-0603-50V-10% -> Seeed-Capacitor:CERAMIC-1NF-1KV-10%-X7R(1206)
- FLASH: device Seeed-Switch:SMD-BUTTON(2P-3.0X2.5X1.2+0.4MM)-B3U-1000P-2P-SMD -> switches:B3U-1000P; SPICEPREFIX (none) -> F
- J6: device SparkFun-Connectors:CONN_08" -> SparkFun-Connectors:CONN_09
- RESET: device Seeed-Switch:SMD-BUTTON(2P-3.0X2.5X1.2+0.4MM)-B3U-1000P-2P-SMD -> switches:B3U-1000P
- U$2: value HLK-PM03 -> HKLPM01; device PowerSocket:HLK-PM03 -> HKLPM01:HKLPM01
- renumbered Q1 to J3Y, Q2 to JY3, U1 to AMS1117
Connections:
- removed net FASE: J1.3, U$2.AC2
- removed net N$2: D3.-, K1.A, K2.A
- new net FASE_IN: R5.1, U$2.AC1, X1-1.KL
- new net VCC_D: D3.-, J6.9, K1.A, K2.A
- net GND: now also FLASH.P$2, RESET.P$2; no longer FLASH.2, RESET.2
- net GPIO0: now also FLASH.P$1; no longer FLASH.1
- net NEUTRAL_IN: now also R5.2, U$2.AC2, X1-2.KL; no longer J1.4, U$2.AC1
- net NEUTRAL_ONE_OUT: now also X1-3.KL; no longer J1.2
- net NEUTRAL_TWO_OUT: now also X1-4.KL; no longer J1.1
- net RESET: now also RESET.P$1; no longer RESET.1
Other:
- note added: "REV3.1"
- note removed: "REV1"
