File: PCB/OnOnfre_dual_mola_ssr_rev3.2/OnOnfre_dual_mola_ssr_rev3.2.brd (EAGLE design)
At the start: 44.4 x 47.7 mm, 24 parts, among them J3Y S8050, J6 8p, J7 8p, K1 OMRON-G3MB-202P-SSR2, K2 OMRON-G3MB-202P-SSR2, U2 esp12

Commit message: resolvido a troca na label dos pinos 04 e 05
Parts:
- removed J6: 8p, SparkFun-Connectors:1X08
- added J1: (no value), SparkFun-Connectors:1X09
Connections:
- removed net N$2: D3.2, K1.3, K2.3
- new net 5V: D3.2, J1.9, K1.3, K2.3
- net GND: now also J1.1; no longer J6.1
- net GPIO0: now also J1.4; no longer J6.4
- net GPIO02: now also J1.3; no longer J6.3
- net GPIO04: now also J1.6; no longer J6.6
- net GPIO05: now also J1.5; no longer J6.5
- net GPIO15: now also J1.2; no longer J6.2
- net RX: now also J1.7; no longer J6.7
- net TX: now also J1.8; no longer J6.8
Routing:
- net 5V: track 0.00 -> 53.2 mm, vias 0 -> 1
- net N$2: track 49.4 -> 0.00 mm, vias 1 -> 0
- net GPIO02: track 2.85 -> 3.62 mm
