File: PCB/OnOnfre_dual_mola_ssr_rev3.2/OnOnfre_dual_mola_ssr_rev3.2.sch (EAGLE design)
At the start: 24 parts, among them J3Y S8050, J6 8p, J7 8p, K1 OMRON-G3MB-202P-SSR2, K2 OMRON-G3MB-202P-SSR2, U2 esp12

Commit message: resolvido a troca na label dos pinos 04 e 05
Parts:
- removed J6: 8p, SparkFun-Connectors:CONN_08"
- added J1: (no value), SparkFun-Connectors:CONN_09
Connections:
- removed net N$2: D3.-, K1.A, K2.A
- new net 5V: D3.-, J1.9, K1.A, K2.A
- net GND: now also J1.1; no longer J6.1
- net GPIO0: now also J1.4; no longer J6.4
- net GPIO02: now also J1.3; no longer J6.3
- net GPIO04: now also J1.6; no longer J6.6
- net GPIO05: now also J1.5; no longer J6.5
- net GPIO15: now also J1.2; no longer J6.2
- net RX: now also J1.7; no longer J6.7
- net TX: now also J1.8; no longer J6.8
Changed lines of the file:
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@@
 <part name="JY3" library="semicon-smd-ipc" library_urn="urn:adsk.eagle:library:353" deviceset="NPN-TRANSISTOR_" device="SOT23" package3d_urn="urn:adsk.eagle:package:26310/1" value="S8050 "/>
 <part name="R1" library="resistor" library_urn="urn:adsk.eagle:library:348" deviceset="R-EU_" device="R0603" package3d_urn="urn:adsk.eagle:package:26057/1" value="10k"/>
-<part name="J6" library="SparkFun-Connectors" library_urn="urn:adsk.eagle:library:513" deviceset="CONN_08" device="&quot;" package3d_urn="urn:adsk.eagle:package:38138/1" value="8p"/>
 <part name="J7" library="SparkFun-Connectors" library_urn="urn:adsk.eagle:library:513" deviceset="CONN_08" device="&quot;" package3d_urn="urn:adsk.eagle:package:38138/1" value="8p"/>
 <part name="RESET" library="switches" deviceset="B3U" device="-1000P" value="B3U-1000P-2P-SMD"/>
@@
 <part name="R5" library="varistor" library_urn="urn:adsk.eagle:library:410" deviceset="VARISTOR" device="S07K230" package3d_urn="urn:adsk.eagle:package:30547/1"/>
 <part name="U$1" library="4po" deviceset="4P" device="4P"/>
+<part name="J1" library="SparkFun-Connectors" library_urn="urn:adsk.eagle:library:513" deviceset="CONN_09" device="" package3d_urn="urn:adsk.eagle:package:38153/1"/>
 </parts>
 <sheets>
@@
 </instance>
 <instance part="R1" gate="G$1" x="106.68" y="50.8" rot="R180"/>
-<instance part="J6" gate="G$1" x="124.46" y="160.02"/>
 <instance part="J7" gate="G$1" x="124.46" y="132.08"/>
 <instance part="RESET" gate="G$1" x="58.42" y="93.98"/>
@@
 <instance part="R5" gate="G$1" x="195.58" y="142.24" rot="R90"/>
 <instance part="U$1" gate="G$1" x="7.62" y="10.16"/>
+<instance part="J1" gate="G$1" x="116.84" y="162.56"/>
 </instances>
 <busses>
@@
 </segment>
 <segment>
-<pinref part="J6" gate="G$1" pin="1"/>
-<wire x1="129.54" y1="152.4" x2="144.78" y2="152.4" width="0.1524" layer="91"/>
+<wire x1="127" y1="152.4" x2="144.78" y2="152.4" width="0.1524" layer="91"/>
 <label x="144.78" y="152.4" size="1.778" layer="95" xref="yes"/>
+<pinref part="J1" gate="G$1" pin="1"/>
 </segment>
 <segment>
@@
 </segment>
 <segment>
-<pinref part="J6" gate="G$1" pin="4"/>
-<wire x1="129.54" y1="160.02" x2="132.08" y2="160.02" width="0.1524" layer="91"/>
+<wire x1="127" y1="160.02" x2="132.08" y2="160.02" width="0.1524" layer="91"/>
 <label x="132.08" y="160.02" size="1.778" layer="95" xref="yes"/>
+<pinref part="J1" gate="G$1" pin="4"/>
 </segment>
 <segment>
@@
 </segment>
 </net>
-<net name="N$2" class="0">
+<net name="5V" class="0">
 <segment>
 <pinref part="D3" gate="G$1" pin="-"/>
@@
 <junction x="129.54" y="66.04"/>
 </segment>
+<segment>
+<pinref part="J1" gate="G$1" pin="9"/>
+<wire x1="127" y1="172.72" x2="147.32" y2="172.72" width="0.1524" layer="91"/>
+<label x="147.32" y="172.72" size="1.778" layer="95" xref="yes"/>
+</segment>
 </net>
 <net name="N$7" class="0">
@@
 </segment>
 <segment>
-<pinref part="J6" gate="G$1" pin="7"/>
-<wire x1="129.54" y1="167.64" x2="144.78" y2="167.64" width="0.1524" layer="91"/>
+<wire x1="127" y1="167.64" x2="144.78" y2="167.64" width="0.1524" layer="91"/>
 <label x="144.78" y="167.64" size="1.778" layer="95" xref="yes"/>
+<pinref part="J1" gate="G$1" pin="7"/>
 </segment>
 </net>
@@
 </segment>
 <segment>
-<pinref part="J6" gate="G$1" pin="6"/>
-<wire x1="129.54" y1="165.1" x2="132.08" y2="165.1" width="0.1524" layer="91"/>
+<wire x1="127" y1="165.1" x2="132.08" y2="165.1" width="0.1524" layer="91"/>
 <label x="132.08" y="165.1" size="1.778" layer="95" xref="yes"/>
+<pinref part="J1" gate="G$1" pin="6"/>
 </segment>
 <segment>
@@
 </segment>
 <segment>
-<pinref part="J6" gate="G$1" pin="5"/>
-<wire x1="129.54" y1="162.56" x2="144.78" y2="162.56" width="0.1524" layer="91"/>
+<wire x1="127" y1="162.56" x2="144.78" y2="162.56" width="0.1524" layer="91"/>
 <label x="144.78" y="162.56" size="1.778" layer="95" xref="yes"/>
+<pinref part="J1" gate="G$1" pin="5"/>
 </segment>
 <segment>
@@
 </segment>
 <segment>
-<pinref part="J6" gate="G$1" pin="3"/>
-<wire x1="129.54" y1="157.48" x2="144.78" y2="157.48" width="0.1524" layer="91"/>
+<wire x1="127" y1="157.48" x2="144.78" y2="157.48" width="0.1524" layer="91"/>
 <label x="144.78" y="157.48" size="1.778" layer="95" xref="yes"/>
+<pinref part="J1" gate="G$1" pin="3"/>
 </segment>
 </net>
@@
 <net name="TX" class="0">
 <segment>
-<pinref part="J6" gate="G$1" pin="8"/>
-<wire x1="129.54" y1="170.18" x2="132.08" y2="170.18" width="0.1524" layer="91"/>
+<wire x1="127" y1="170.18" x2="132.08" y2="170.18" width="0.1524" layer="91"/>
 <label x="132.08" y="170.18" size="1.778" layer="95" xref="yes"/>
+<pinref part="J1" gate="G$1" pin="8"/>
 </segment>
 <segment>
@@
 <net name="GPIO15" class="0">
 <segment>
-<pinref part="J6" gate="G$1" pin="2"/>
-<wire x1="129.54" y1="154.94" x2="132.08" y2="154.94" width="0.1524" layer="91"/>
+<wire x1="127" y1="154.94" x2="132.08" y2="154.94" width="0.1524" layer="91"/>
 <label x="132.08" y="154.94" size="1.778" layer="95" xref="yes"/>
-</segment>
-<segment>
+<pinref part="J1" gate="G$1" pin="2"/>
+</segment>
+<segment>
