File: PCB/OnOnfre_dual_mola_ssr_rev3.4/OnOnfre_dual_mola_ssr_rev3.4.sch (EAGLE design)
At the start: 24 parts, among them J3Y S8050, J7 8p, K1 OMRON-G3MB-202P-SSR2, K2 OMRON-G3MB-202P-SSR2, U2 esp12

Commit message: Rev 3.4, alteração de labels e numero de pinos
Connections:
- net GPIO04: now also J1.5, R4.1; no longer J1.6, R1.1
- net GPIO05: now also J1.6, R1.1; no longer J1.5, R4.1
Other:
- note removed: "REV1"
Changed lines of the file:
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@@
 <text x="175.26" y="167.64" size="6.4516" layer="95">BH ON OFRE 12</text>
 <text x="53.34" y="157.48" size="5.08" layer="95">ESP8266-12</text>
-<text x="175.26" y="160.02" size="6.4516" layer="95">REV1</text>
 </plain>
 <instances>
@@
 <wire x1="203.2" y1="142.24" x2="195.58" y2="137.16" width="0.1524" layer="91"/>
 <pinref part="R5" gate="G$1" pin="2"/>
-<wire x1="195.58" y1="137.16" x2="180.34" y2="142.24" width="0.1524" layer="91"/>
+<wire x1="195.58" y1="137.16" x2="182.88" y2="137.16" width="0.1524" layer="91"/>
 <junction x="195.58" y="137.16"/>
-<label x="180.34" y="142.24" size="1.778" layer="95" rot="R180"/>
+<label x="182.88" y="137.16" size="1.778" layer="95" rot="R180" xref="yes"/>
 </segment>
 <segment>
@@
 </segment>
 <segment>
-<label x="33.02" y="7.62" size="1.778" layer="95" xref="yes"/>
-<wire x1="10.16" y1="10.16" x2="33.02" y2="7.62" width="0.1524" layer="91"/>
+<label x="22.86" y="10.16" size="1.778" layer="95" xref="yes"/>
+<wire x1="10.16" y1="10.16" x2="22.86" y2="10.16" width="0.1524" layer="91"/>
 <pinref part="U$1" gate="G$1" pin="P4"/>
 <junction x="10.16" y="10.16"/>
@@
 <segment>
 <pinref part="U2" gate="G$1" pin="GPIO4"/>
+<wire x1="86.36" y1="144.78" x2="88.9" y2="144.78" width="0.1524" layer="91"/>
+<label x="88.9" y="144.78" size="1.778" layer="95" xref="yes"/>
+</segment>
+<segment>
+<wire x1="127" y1="162.56" x2="144.78" y2="162.56" width="0.1524" layer="91"/>
+<label x="144.78" y="162.56" size="1.778" layer="95" xref="yes"/>
+<pinref part="J1" gate="G$1" pin="5"/>
+</segment>
+<segment>
+<pinref part="R4" gate="G$1" pin="1"/>
+<wire x1="111.76" y1="78.74" x2="116.84" y2="78.74" width="0.1524" layer="91"/>
+<label x="116.84" y="78.74" size="1.778" layer="95" xref="yes"/>
+</segment>
+</net>
+<net name="GPIO05" class="0">
+<segment>
+<pinref part="U2" gate="G$1" pin="GPIO5"/>
 <wire x1="86.36" y1="147.32" x2="88.9" y2="147.32" width="0.1524" layer="91"/>
 <label x="88.9" y="147.32" size="1.778" layer="95" xref="yes"/>
@@
 <wire x1="111.76" y1="50.8" x2="116.84" y2="50.8" width="0.1524" layer="91"/>
 <label x="116.84" y="50.8" size="1.778" layer="95" xref="yes"/>
-</segment>
-</net>
-<net name="GPIO05" class="0">
-<segment>
-<pinref part="U2" gate="G$1" pin="GPIO5"/>
-<wire x1="86.36" y1="144.78" x2="88.9" y2="144.78" width="0.1524" layer="91"/>
-<label x="88.9" y="144.78" size="1.778" layer="95" xref="yes"/>
-</segment>
-<segment>
-<wire x1="127" y1="162.56" x2="144.78" y2="162.56" width="0.1524" layer="91"/>
-<label x="144.78" y="162.56" size="1.778" layer="95" xref="yes"/>
-<pinref part="J1" gate="G$1" pin="5"/>
-</segment>
-<segment>
-<pinref part="R4" gate="G$1" pin="1"/>
-<wire x1="111.76" y1="78.74" x2="116.84" y2="78.74" width="0.1524" layer="91"/>
-<label x="116.84" y="78.74" size="1.778" layer="95" xref="yes"/>
 </segment>
 </net>
@@
 <wire x1="195.58" y1="147.32" x2="180.34" y2="147.32" width="0.1524" layer="91"/>
 <junction x="195.58" y="147.32"/>
-<label x="180.34" y="147.32" size="1.778" layer="95" rot="R180"/>
-</segment>
-<segment>
+<label x="180.34" y="147.32" size="1.778" layer="95" rot="R180" xref="yes"/>
+</segment>
+<segment>
