File: PCB/OnOnfre_dual_parafuso_estores_beta/OnOnfre_dual_parafuso_estores_beta.sch (EAGLE design)
At the start: 41 parts, among them IC4 HLW8012, J7 8p, Q3 2N7002, Q4 2N7002, U2 esp12

Commit message: estores e tomada em progresso
Parts:
- removed C41, C42: 33nF, xose:C-EU0805
- removed C43, C45: 100nF, xose:C-EU0805
- removed C44: 1uF, xose:C-EU0805
- removed IC4: HLW8012, xose:HLW8012
- removed Q3, Q4: 2N7002, xose:MOSFET-NREFLOW
- removed R31, R43, R44, R50: 1K, xose:RESISTOR0805
- removed R32, R45, R47, R49: 10K, xose:RESISTOR0805
- removed R41: 0.001R, xose:RESISTOR2512
- removed R42: 0R, xose:RESISTOR1206
- removed R46, R48: 15K, xose:RESISTOR0805
- removed R51, R52, R53, R54, R55: 470K, xose:RESISTOR0805
- removed RLY1: SRD-05VDC-SL-C, Spark:RELAYSONGLE
- added D2: 1N4007, Seeed-Diode:DIODE-GEN-PURPOSE-1KV-1A(DO-214AC)
- added D3: 1N4004, Seeed-Diode:DIODE-GEN-PURPOSE-1KV-1A(DO-214AC)
- added F1: FUSE 2A, SparkFun-Fuses:PPTC_PTH
- added J3Y, JY3: S8050, semicon-smd-ipc:NPN-TRANSISTOR_SOT23
- added R1, R2, R3, R4: 10k, resistor:R-EU_R0603
- added U$1, U$3: HF46F, HF46F:HF46F
- D1: value 1N4148 -> 1N4007; device xose:DIODE -> Seeed-Diode:DIODE-GEN-PURPOSE-1KV-1A(DO-214AC)
Connections:
- removed net GPIO5: Q4.G
- removed net LINE_IN: R41.2, R43.2, R5.1, U$2.AC1, X1-1.KL
- removed net LINE_R: R41.1, R42.2, R44.2, RLY1.MAIN
- removed net N$10: IC4.SEL, Q4.D, R49.1
- removed net N$11: IC4.CF1, R45.2
- removed net N$12: C41.2, IC4.V1P, R43.1
- removed net N$14: C42.2, IC4.V1N, R44.1
- removed net N$15: R53.1, R54.1
- removed net N$16: R54.2, R55.2
- removed net N$2: IC4.CF, R47.2
- removed net N$4: D1.A, Q3.D, RLY1.COIL2
- removed net N$5: Q3.G, R31.2, R32.2
- removed net N$6: R51.1, R52.1
- removed net N$8: R52.2, R53.2
- removed net NC: RLY1.NC, X1-4.KL
- removed net NO: RLY1.NO, X1-3.KL
- removed net V2P: C45.2, IC4.V2P, R50.2, R55.1
- new net FASE_IN: R5.1, U$2.AC1, X1-1.KL
- new net N$1: D1.+, J3Y.C, U$1.C2
- new net N$13: JY3.B, R1.2, R2.2
- new net N$7: J3Y.B, R3.2, R4.2
- new net N$9: D2.+, JY3.C, U$3.C2
- new net NEUTRAL_IN_FUSED: F1.2, U$1.L2, U$3.L2
- new net NEUTRAL_ONE_OUT: U$3.L1, X1-3.KL
- new net NEUTRAL_TWO_OUT: U$1.L1, X1-4.KL
- net 5V: now also D1.-, D2.-, D3.-, U$1.C1, U$3.C1; no longer C43.2, C44.2, D1.C, IC4.VDD, R49.2, RLY1.COIL1
- net GND: now also J3Y.E, JY3.E, R2.1, R3.1; no longer C41.1, C42.1, C43.1, C44.1, C45.1, IC4.GND, Q3.S, Q4.S, R32.1, R42.1, R46.1, R48.1, R50.1
- net GPIO04: now also R4.1
- net GPIO05: now also R1.1
- net GPIO12: no longer R31.1
- net GPIO13: no longer R45.1, R46.2
- net GPIO14: no longer R47.1, R48.2
- net NEUTRAL_IN: now also F1.1; no longer R51.2
- net VCC: now also D3.+
Other:
- note added: "BH ON OFRE 12"
- note removed: "ADICIONAR FUSIVEL DE FUSÃO RAPIDA E FUSIVEL TERMICO DE 73 Graus 10A"
- note removed: "Alimentação"
- note removed: "GPIOS"
- note removed: "Medição de consumo"
- note removed: "Microcontrolador"
- note removed: "Protecção"
- moved on the sheet: AMS1117, C4, FLASH, J1, J7, R10, R11, R5, R8, R9, RESET, U$2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

Commit message: remoção do OTA Arduino e adição de OTA via Web
Parts:
- removed R5: VARISTORS07K230, varistor:VARISTORS07K230
Connections:
- removed net FASE_IN: R5.1, U$2.AC1, X1-1.KL
- new net LINE_IN: U$2.AC2, X1-1.KL
- net NEUTRAL_IN: now also U$2.AC1; no longer R5.2, U$2.AC2
- net NEUTRAL_IN_FUSED: now also U$1.L1, U$3.L1; no longer U$1.L2, U$3.L2
- net NEUTRAL_ONE_OUT: now also U$1.L2; no longer U$3.L1
- net NEUTRAL_TWO_OUT: now also U$3.L2; no longer U$1.L1
Changed lines of the file:
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@@
 <part name="AMS1117" library="SparkFun-IC-Power" library_urn="urn:adsk.eagle:library:526" deviceset="V_REG_LM1117" device="SOT223" package3d_urn="urn:adsk.eagle:package:39069/1" value="LM1117"/>
 <part name="FLASH" library="switches" deviceset="B3U" device="-1000P" value="B3U-1000P-2P-SMD"/>
-<part name="R5" library="varistor" library_urn="urn:adsk.eagle:library:410" deviceset="VARISTOR" device="S07K230" package3d_urn="urn:adsk.eagle:package:30547/1"/>
 <part name="J1" library="SparkFun-Connectors" library_urn="urn:adsk.eagle:library:513" deviceset="CONN_09" device="" package3d_urn="urn:adsk.eagle:package:38153/1"/>
 <part name="X1" library="con-wago-500" library_urn="urn:adsk.eagle:library:195" deviceset="W237-4" device="" package3d_urn="urn:adsk.eagle:package:10695/1"/>
@@
 <instance part="AMS1117" gate="G$1" x="167.64" y="111.76"/>
 <instance part="FLASH" gate="G$1" x="58.42" y="109.22"/>
-<instance part="R5" gate="G$1" x="195.58" y="142.24" rot="R90"/>
 <instance part="J1" gate="G$1" x="116.84" y="162.56"/>
 <instance part="X1" gate="-1" x="12.7" y="25.4"/>
@@
 </segment>
 <segment>
-<pinref part="U$2" gate="G$1" pin="AC2"/>
-<wire x1="203.2" y1="142.24" x2="195.58" y2="137.16" width="0.1524" layer="91"/>
-<pinref part="R5" gate="G$1" pin="2"/>
-<wire x1="195.58" y1="137.16" x2="182.88" y2="137.16" width="0.1524" layer="91"/>
-<junction x="195.58" y="137.16"/>
-<label x="182.88" y="137.16" size="1.778" layer="95" rot="R180" xref="yes"/>
-</segment>
-<segment>
 <label x="27.94" y="20.32" size="1.778" layer="95" xref="yes"/>
 <pinref part="X1" gate="-2" pin="KL"/>
 <wire x1="17.78" y1="20.32" x2="27.94" y2="20.32" width="0.1524" layer="91"/>
 </segment>
+<segment>
+<pinref part="U$2" gate="G$1" pin="AC1"/>
+<wire x1="203.2" y1="147.32" x2="180.34" y2="147.32" width="0.1524" layer="91"/>
+<label x="180.34" y="147.32" size="1.778" layer="95" rot="R180" xref="yes"/>
+</segment>
 </net>
 <net name="NEUTRAL_TWO_OUT" class="1">
@@
 </segment>
 <segment>
-<pinref part="U$1" gate="G$1" pin="L1"/>
-<wire x1="71.12" y1="58.42" x2="66.04" y2="58.42" width="0.1524" layer="91"/>
-<label x="66.04" y="58.42" size="1.778" layer="95" rot="R180" xref="yes"/>
+<wire x1="76.2" y1="35.56" x2="78.74" y2="35.56" width="0.1524" layer="91"/>
+<label x="78.74" y="35.56" size="1.778" layer="95" xref="yes"/>
+<pinref part="U$3" gate="G$1" pin="L2"/>
 </segment>
 </net>
 <net name="NEUTRAL_ONE_OUT" class="1">
-<segment>
-<wire x1="63.5" y1="35.56" x2="68.58" y2="35.56" width="0.1524" layer="91"/>
-<label x="63.5" y="35.56" size="1.778" layer="95" rot="R180" xref="yes"/>
-<pinref part="U$3" gate="G$1" pin="L1"/>
-</segment>
 <segment>
 <label x="22.86" y="15.24" size="1.778" layer="95" xref="yes"/>
 <pinref part="X1" gate="-3" pin="KL"/>
 <wire x1="17.78" y1="15.24" x2="22.86" y2="15.24" width="0.1524" layer="91"/>
+</segment>
+<segment>
+<wire x1="78.74" y1="58.42" x2="81.28" y2="58.42" width="0.1524" layer="91"/>
+<label x="81.28" y="58.42" size="1.778" layer="95" xref="yes"/>
+<pinref part="U$1" gate="G$1" pin="L2"/>
 </segment>
 </net>
@@
 </segment>
 <segment>
-<wire x1="76.2" y1="35.56" x2="78.74" y2="35.56" width="0.1524" layer="91"/>
-<label x="78.74" y="35.56" size="1.778" layer="95" xref="yes"/>
-<pinref part="U$3" gate="G$1" pin="L2"/>
-</segment>
-<segment>
-<wire x1="78.74" y1="58.42" x2="81.28" y2="58.42" width="0.1524" layer="91"/>
-<label x="81.28" y="58.42" size="1.778" layer="95" xref="yes"/>
-<pinref part="U$1" gate="G$1" pin="L2"/>
+<pinref part="U$1" gate="G$1" pin="L1"/>
+<wire x1="71.12" y1="58.42" x2="66.04" y2="58.42" width="0.1524" layer="91"/>
+<label x="66.04" y="58.42" size="1.778" layer="95" rot="R180" xref="yes"/>
+</segment>
+<segment>
+<wire x1="63.5" y1="35.56" x2="68.58" y2="35.56" width="0.1524" layer="91"/>
+<label x="63.5" y="35.56" size="1.778" layer="95" rot="R180" xref="yes"/>
+<pinref part="U$3" gate="G$1" pin="L1"/>
 </segment>
 </net>
@@
 </segment>
 </net>
-<net name="FASE_IN" class="1">
-<segment>
-<pinref part="U$2" gate="G$1" pin="AC1"/>
-<wire x1="203.2" y1="147.32" x2="195.58" y2="147.32" width="0.1524" layer="91"/>
-<pinref part="R5" gate="G$1" pin="1"/>
-<wire x1="195.58" y1="147.32" x2="180.34" y2="147.32" width="0.1524" layer="91"/>
-<junction x="195.58" y="147.32"/>
-<label x="180.34" y="147.32" size="1.778" layer="95" rot="R180" xref="yes"/>
-</segment>
-<segment>
+<net name="LINE_IN" class="1">
+<segment>
+<pinref part="U$2" gate="G$1" pin="AC2"/>
+<wire x1="203.2" y1="142.24" x2="195.58" y2="137.16" width="0.1524" layer="91"/>
+<wire x1="195.58" y1="137.16" x2="182.88" y2="137.16" width="0.1524" layer="91"/>
+<label x="182.88" y="137.16" size="1.778" layer="95" rot="R180" xref="yes"/>
+</segment>
+<segment>

Commit message: Rev3.5 Parafuso
Parts:
- F1: value FUSE 2A -> FUSE
Changed lines of the file:
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@@
 </classes>
 <parts>
-<part name="F1" library="SparkFun-Fuses" library_urn="urn:adsk.eagle:library:517" deviceset="PPTC" device="_PTH" package3d_urn="urn:adsk.eagle:package:38574/1" value="FUSE 2A"/>
+<part name="F1" library="SparkFun-Fuses" library_urn="urn:adsk.eagle:library:517" deviceset="PPTC" device="_PTH" package3d_urn="urn:adsk.eagle:package:38574/1" value="FUSE "/>
 <part name="J3Y" library="semicon-smd-ipc" library_urn="urn:adsk.eagle:library:353" deviceset="NPN-TRANSISTOR_" device="SOT23" package3d_urn="urn:adsk.eagle:package:26310/1" value="S8050 "/>
 <part name="R4" library="resistor" library_urn="urn:adsk.eagle:library:348" deviceset="R-EU_" device="R0603" package3d_urn="urn:adsk.eagle:package:26057/1" value="10k"/>
