File: PCB/OnOnfre_dual_parafuso_ssr_rev4/OnOnfre_dual_parafuso_ssr.sch (EAGLE design)
At the start: 24 parts, among them J3Y S8050, J7 8p, K1 OMRON-G3MB-202P-SSR2, K2 OMRON-G3MB-202P-SSR2, U2 esp12

Commit message: no message
Parts:
- removed J1: (no value), SparkFun-Connectors:CONN_09
- removed J7: 8p, SparkFun-Connectors:CONN_08"
- added C1, C2: 22uF, Seeed-Capacitor:CERAMIC-1NF-1KV-10%-X7R(1206)
- added C3: 100uF, Seeed-Capacitor:CERAMIC-1NF-1KV-10%-X7R(1206)
- added C5: (no value), rcl:C-EU102-054X133
- added L1: (no value), inductor-neosid:ZD60820510
- C4: value 100NF -> 100uF
Connections:
- removed net FASE_IN: R5.1, U$2.AC1, X1-1.KL
- removed net NEUTRAL_IN: F1.1, R5.2, U$2.AC2, X1-2.KL
- removed net NEUTRAL_IN_FUSED: F1.2, K1.DS2, K2.DS2
- new net EMI_LINE: L1.2, U$2.AC2
- new net EMI_NEUTRAL: L1.1, U$2.AC1
- new net LINE: F1.1, X1-1.KL
- new net N$2: C5.1, F1.2, L1.3, R5.2
- new net NEUTRAL: C5.2, K1.DS2, K2.DS2, L1.4, R5.1, X1-2.KL
- net 3V3: now also C1.1; no longer J7.1
- net 5V: no longer J1.9
- net ADC: no longer J7.7
- net CH_PD: no longer J7.6
- net GND: now also C1.2, C2.2, C3.2; no longer J1.1
- net GPIO0: no longer J1.4
- net GPIO02: no longer J1.3
- net GPIO04: no longer J1.5
- net GPIO05: no longer J1.6
- net GPIO12: no longer J7.3
- net GPIO13: no longer J7.2
- net GPIO14: no longer J7.4
- net GPIO15: no longer J1.2
- net GPIO16: no longer J7.5
- net RESET: no longer J7.8
- net RX: no longer J1.7
- net TX: no longer J1.8
- net VCC: now also C2.1, C3.1
Other:
- moved on the sheet: C4, F1, R5, U$2
