File: OnOfre EasyLight/PCB_OnOnfre_Easy_Light/OnOnfre_Easy_Light_dev.sch (EAGLE design)
At the start: 27 parts, among them J3Y S8050, K1 OMRON-G3MB-202P-SSR2, K2 OMRON-G3MB-202P-SSR2, U2 esp12

Commit message: no message
Parts:
- removed FLASH: B3U-1000P-2P-SMD, switches:B3U-1000P
- added A0, GPIO14, GPIO16: BM03B-SRSS-TB, con-jst2:BM03B-SRSS-TB
- added C6: 100nf, Seeed-Capacitor:CERAMIC-100NF-50V-10%-X7R(0603)
- added D1, D2, D4: (no value), diode:DIODE-SOD323-R
- added F2: (no value), adafruit:PTCFUSE-1812
- added FTDI: BM05B-SRSS-TB, con-jst2:BM05B-SRSS-TB
- added R6: 100k, resistor:R-EU_R0603
- added R7: 220k, resistor:R-EU_R0603
- added SWITCHS: BM04B-SRSS-TB, con-jst2:BM04B-SRSS-TB
- C1, C2: value 22uF -> 22uf
- C3, C4: value 100uF -> 100uf
- D3: value 1N4004 -> 1N4007
- F1: value 0.5A -> (none); device SparkFun-Fuses:PPTC_PTH -> adafruit:PTCFUSE-1812
Connections:
- removed net 3V3: AMS1117.OUT, C1.1, C4.1, R10.2, R8.2, R9.2, U2.VCC
- removed net VCC: AMS1117.IN, C2.1, C3.1, D3.+, U$2.+VO
- new net A0: A0-3.S, R7.2
- new net DTR: D2.C, FTDI-5.S
- new net LIVE_FUSED: F1.2, K1.DS1, K2.DS1
- new net N$3: D1.C, FTDI-3.S
- new net N$4: C6.2, D2.A, D4.C
- new net VCC_1: AMS1117.IN, C2.1, C3.1, D3.+, FTDI-1.S, U$2.+VO
- new net VCC_2: A0-1.S, AMS1117.OUT, C1.1, C4.1, GPIO14-1.S, GPIO16-1.S, R10.2, R8.2, R9.2, SWITCHS-1.S, U2.VCC
- net ADC: now also R6.2, R7.1
- net CH_PD: now also C6.1
- net GND: now also A0-2.S, FTDI-2.S, GPIO14-2.S, GPIO16-2.S, R6.1, SWITCHS-2.S; no longer FLASH.P$2
- net GPIO0: no longer FLASH.P$1
- net GPIO12: now also SWITCHS-4.S
- net GPIO13: now also SWITCHS-3.S
- net GPIO14: now also GPIO14-3.S
- net GPIO16: now also GPIO16-3.S
- net LIVE: now also F2.1; no longer K1.DS1, K2.DS1
- net N$2: now also F2.2; no longer F1.2
- net RESET: now also D4.A
- net RX: now also D1.A
- net TX: now also FTDI-4.S
Other:
- note added: "CONTROL BUTTONS"
- note added: "EXTRA GPIOS"
- note added: "FTDI"
- note added: "MICRO CONTROLLER"
- note added: "OnOfre - EASY LIGHT"
- note added: "POWER SUPPLY"
- note added: "RELAYS"
- note added: "SWITCHS"
- note removed: "BH ON OFRE 12"
- note removed: "ESP8266-12"
- moved on the sheet: AMS1117, C1, C2, C3, C4, C5, D3, J3Y, JY3, K1, K2, L1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

Commit message: versão beta 1
Parts:
- removed L1: (no value), inductor-neosid:ZD60820510
- added L2: (no value), inductor-onofre:ZD60820510
Connections:
- net EMI_LIVE: now also L2.4; no longer L1.2
- net EMI_NEUTRAL: now also L2.3; no longer L1.1
- net N$2: now also L2.1; no longer L1.3
- net NEUTRAL: now also L2.2; no longer L1.4
Changed lines of the file:
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@@
 <part name="C3" library="Seeed-Capacitor" library_urn="urn:adsk.eagle:library:464" deviceset="CERAMIC-1NF-1KV-10%-X7R?(1206)" device="" package3d_urn="urn:adsk.eagle:package:32384/1" value="100uf"/>
 <part name="C5" library="rcl" library_urn="urn:adsk.eagle:library:334" deviceset="C-EU" device="102-054X133" package3d_urn="urn:adsk.eagle:package:23649/1"/>
-<part name="L1" library="inductor-neosid" library_urn="urn:adsk.eagle:library:241" deviceset="ZD60820510" device="" package3d_urn="urn:adsk.eagle:package:14675/1"/>
 <part name="D1" library="diode" library_urn="urn:adsk.eagle:library:210" deviceset="DIODE-" device="SOD323-R" package3d_urn="urn:adsk.eagle:package:43437/1"/>
 <part name="D2" library="diode" library_urn="urn:adsk.eagle:library:210" deviceset="DIODE-" device="SOD323-R" package3d_urn="urn:adsk.eagle:package:43437/1"/>
@@
 <part name="SUPPLY2" library="SparkFun-PowerSymbols" library_urn="urn:adsk.eagle:library:530" deviceset="VCC_1" device=""/>
 <part name="SUPPLY3" library="SparkFun-PowerSymbols" library_urn="urn:adsk.eagle:library:530" deviceset="VCC_2" device=""/>
+<part name="L2" library="inductor-onofre" deviceset="ZD60820510" device=""/>
 </parts>
 <sheets>
@@
 <instance part="C3" gate="G$1" x="297.18" y="101.6" rot="R270"/>
 <instance part="C5" gate="G$1" x="292.1" y="154.94"/>
-<instance part="L1" gate="G$1" x="304.8" y="154.94" rot="R180"/>
 <instance part="D1" gate="G$1" x="33.02" y="134.62"/>
 <instance part="D2" gate="G$1" x="33.02" y="129.54"/>
@@
 <instance part="SUPPLY2" gate="G$2" x="332.74" y="116.84"/>
 <instance part="SUPPLY3" gate="G$1" x="330.2" y="106.68"/>
+<instance part="L2" gate="G$1" x="307.34" y="157.48"/>
 </instances>
 <busses>
@@
 <wire x1="292.1" y1="149.86" x2="292.1" y2="147.32" width="0.1524" layer="91"/>
 <wire x1="299.72" y1="147.32" x2="292.1" y2="147.32" width="0.1524" layer="91"/>
-<pinref part="L1" gate="G$1" pin="4"/>
 <wire x1="302.26" y1="154.94" x2="302.26" y2="147.32" width="0.1524" layer="91"/>
 <wire x1="302.26" y1="147.32" x2="299.72" y2="147.32" width="0.1524" layer="91"/>
+<pinref part="L2" gate="G$1" pin="2"/>
 </segment>
 <segment>
@@
 <wire x1="292.1" y1="157.48" x2="292.1" y2="162.56" width="0.1524" layer="91"/>
 <wire x1="299.72" y1="162.56" x2="292.1" y2="162.56" width="0.1524" layer="91"/>
-<pinref part="L1" gate="G$1" pin="3"/>
 <wire x1="299.72" y1="162.56" x2="299.72" y2="157.48" width="0.1524" layer="91"/>
 <wire x1="299.72" y1="157.48" x2="302.26" y2="157.48" width="0.1524" layer="91"/>
 <pinref part="F2" gate="G$1" pin="2"/>
+<pinref part="L2" gate="G$1" pin="1"/>
 </segment>
 </net>
 <net name="EMI_NEUTRAL" class="1">
 <segment>
-<pinref part="L1" gate="G$1" pin="1"/>
 <wire x1="309.88" y1="154.94" x2="330.2" y2="154.94" width="0.1524" layer="91"/>
 <label x="330.2" y="154.94" size="1.778" layer="95" xref="yes"/>
+<pinref part="L2" gate="G$1" pin="3"/>
 </segment>
 <segment>
@@
 </segment>
 <segment>
-<pinref part="L1" gate="G$1" pin="2"/>
 <wire x1="309.88" y1="157.48" x2="312.42" y2="157.48" width="0.1524" layer="91"/>
 <label x="312.42" y="157.48" size="1.778" layer="95" xref="yes"/>
-</segment>
-</net>
+<pinref part="L2" gate="G$1" pin="4"/>
+</segment>
+</net>

Commit message: no message
Parts:
- C5: value (none) -> 0.1uf 275v
- D1, D2, D4: value (none) -> B5819W
- F1: value (none) -> 2A
- F2: value (none) -> 0.5A
- L2: value (none) -> 10MH
- X1: value (none) -> 4P
Connections:
- removed net GPIO02: U2.GPIO2
