File: OnOfre DevBoard/PCB_OnOnfre_DevBoard4.1/OnOnfre_DevBoard.sch (EAGLE design)
At the start: 27 parts, among them J3Y S8050, J7 8p, K1 OMRON-G3MB-202P-SSR2, K2 OMRON-G3MB-202P-SSR2, U2 esp12

Commit message: Revert "rev5.0dev"
This reverts commit 2e2358a8c57761c3fa030a0a65c911856fe9a90b.
Parts:
- C1, C2: value 1NF -> 22uF
- C3, C4: value 1NF -> 100uF
- D3: value 1N4007 -> 1N4004
- F1: value 6V/0.75A -> FUSE 2A; device SparkFun-Fuses:PPTC_THREE-QUARTER-AMP -> SparkFun-Fuses:PPTC_PTH
- R5: value 10D391K 390V -> VARISTORS07K230
Connections:
- removed net LIVE: F1.1, R5.1, U$2.AC1, X1-2.KL
- removed net LIVE_FUSED: F1.2, K1.DS1, K2.DS1
- removed net LIVE_ONE_OUT: K2.DS2, X1-3.KL
- removed net LIVE_TWO_OUT: K1.DS2, X1-4.KL
- removed net N$2: U2.VCC
- removed net NEUTRAL: R5.2, U$2.AC2, X1-1.KL
- new net FASE_IN: R5.1, U$2.AC1, X1-1.KL
- new net NEUTRAL_IN: F1.1, R5.2, U$2.AC2, X1-2.KL
- new net NEUTRAL_IN_FUSED: F1.2, K1.DS2, K2.DS2
- new net NEUTRAL_ONE_OUT: K1.DS1, X1-3.KL
- new net NEUTRAL_TWO_OUT: K2.DS1, X1-4.KL
- net 3V3: now also U2.VCC
Other:
- note added: "BH ON OFRE 12"
- note removed: "BH ON OFRE DEV BOARD"
- moved on the sheet: AMS1117, C1, C2, C3, C4, D3, F1, FLASH, J1, J3Y, J7, JY3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
