File: PCB/PCB_OnOnfre_DUAL_4A_beta2/OnOnfre_EasyBlinds_beta2.sch (EAGLE design)
At the start: 27 parts, among them J3Y S8050, J7 8p, K1 OMRON-G3MB-202P-SSR2, K2 OMRON-G3MB-202P-SSR2, U2 esp12

Commit message: beta2 board 5A
Parts:
- removed C1, C2: 22uF, Seeed-Capacitor:CERAMIC-1NF-1KV-10%-X7R(1206)
- removed C3: 100uF, Seeed-Capacitor:CERAMIC-1NF-1KV-10%-X7R(1206)
- removed K1, K2: OMRON-G3MB-202P-SSR2, Omron G3MB 202p SSR:OMRON-G3MB-202P-SSR2
- removed R5: VARISTORS07K230, varistor:VARISTORS07K230
- added D1, D2: 1N4007, Seeed-Diode:DIODE-GEN-PURPOSE-1KV-1A(DO-214AC)
- added U$1, U$3: HF46F, HF46F:HF46F
- C4: value 100uF -> 100NF
- F1: value FUSE 2A -> FUSE
Connections:
- removed net FASE_IN: R5.1, U$2.AC1, X1-1.KL
- new net LINE_IN: U$2.AC2, X1-1.KL
- net 3V3: no longer C1.1
- net 5V: now also D1.-, D2.-, U$1.C1, U$3.C1; no longer K1.A, K2.A
- net GND: no longer C1.2, C2.2, C3.2
- net N$1: now also D1.+, U$1.C2; no longer K1.K
- net N$9: now also D2.+, U$3.C2; no longer K2.K
- net NEUTRAL_IN: now also U$2.AC1; no longer R5.2, U$2.AC2
- net NEUTRAL_IN_FUSED: now also U$1.L1, U$3.L1; no longer K1.DS2, K2.DS2
- net NEUTRAL_ONE_OUT: now also U$1.L2; no longer K1.DS1
- net NEUTRAL_TWO_OUT: now also U$3.L2; no longer K2.DS1
- net VCC: no longer C2.1, C3.1
Other:
- moved on the sheet: C4, D3, J3Y, JY3, R1, R2, R3, R4
