File: PCB/PCB_OnOnfre_DUAL_rev5.0/OnOnfre_DevBoard_rev5.sch (EAGLE design)
At the start: 28 parts, among them J1 9PIN 2.54MM, J3Y S8050, J7 8p, K1 OMRON-G3MB-202P-SSR2, K2 OMRON-G3MB-202P-SSR2, U2 esp12

Commit message: Revert "rev5.1"
This reverts commit eb04db9ecb2416f00214f08c4929ad914bbcba1f.
Parts:
- added D1, D2: 1N4148, diode:DIODE-SOD80C
- added JP1, JP2: (no value), pinhead:PINHD-1X1
Connections:
- net LINE_L: now also JP1.1, JP2.1
- net N$1: now also D1.C
- net N$9: now also D2.C
- net VCC: now also D1.A, D2.A
Other:
- note added: "BH ON OFRE 12"
- note added: "ESP8266-12"
Changed lines of the file:
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@@
 <?xml version="1.0" encoding="utf-8"?>
 <!DOCTYPE eagle SYSTEM "eagle.dtd">
-<eagle version="9.1.3">
+<eagle version="9.2.2">
 <drawing>
 <settings>
@@
 <part name="C3" library="Seeed-Capacitor" library_urn="urn:adsk.eagle:library:464" deviceset="CERAMIC-1NF-1KV-10%-X7R?(1206)" device="" package3d_urn="urn:adsk.eagle:package:32384/1" value="100uF"/>
 <part name="U$1" library="HLK-PM01" deviceset="HLK-PM01" device=""/>
+<part name="JP1" library="pinhead" library_urn="urn:adsk.eagle:library:325" deviceset="PINHD-1X1" device="" package3d_urn="urn:adsk.eagle:package:22485/2"/>
+<part name="JP2" library="pinhead" library_urn="urn:adsk.eagle:library:325" deviceset="PINHD-1X1" device="" package3d_urn="urn:adsk.eagle:package:22485/2"/>
+<part name="D1" library="diode" library_urn="urn:adsk.eagle:library:210" deviceset="DIODE-" device="SOD80C" package3d_urn="urn:adsk.eagle:package:43405/2" value="1N4148"/>
+<part name="D2" library="diode" library_urn="urn:adsk.eagle:library:210" deviceset="DIODE-" device="SOD80C" package3d_urn="urn:adsk.eagle:package:43405/2" value="1N4148"/>
 <part name="F1" library="polyfuse-smd_10" deviceset="?" device="1812L" technology="010"/>
 <part name="R5" library="VARISTORESBH" deviceset="S07K230" device=""/>
@@
 <plain>
 <text x="203.2" y="144.78" size="1.778" layer="95">HLK-PM05</text>
+<text x="175.26" y="167.64" size="6.4516" layer="95">BH ON OFRE 12</text>
+<text x="53.34" y="157.48" size="5.08" layer="95">ESP8266-12</text>
 </plain>
 <instances>
@@
 <instance part="U$1" gate="G$1" x="223.52" y="144.78" smashed="yes">
 <attribute name="NAME" x="213.36" y="137.16" size="1.778" layer="94"/>
+</instance>
+<instance part="JP1" gate="G$1" x="25.4" y="58.42" smashed="yes" rot="R180">
+<attribute name="NAME" x="31.75" y="55.245" size="1.778" layer="95" rot="R180"/>
+<attribute name="VALUE" x="31.75" y="63.5" size="1.778" layer="96" rot="R180"/>
+</instance>
+<instance part="JP2" gate="G$1" x="25.4" y="33.02" smashed="yes" rot="R180">
+<attribute name="NAME" x="31.75" y="29.845" size="1.778" layer="95" rot="R180"/>
+<attribute name="VALUE" x="31.75" y="38.1" size="1.778" layer="96" rot="R180"/>
+</instance>
+<instance part="D1" gate="G$1" x="83.82" y="68.58" smashed="yes" rot="R90">
+<attribute name="NAME" x="83.3374" y="71.12" size="1.778" layer="95" rot="R90"/>
+<attribute name="VALUE" x="86.1314" y="71.12" size="1.778" layer="96" rot="R90"/>
+</instance>
+<instance part="D2" gate="G$1" x="83.82" y="43.18" smashed="yes" rot="R90">
+<attribute name="NAME" x="83.3374" y="45.72" size="1.778" layer="95" rot="R90"/>
+<attribute name="VALUE" x="86.1314" y="45.72" size="1.778" layer="96" rot="R90"/>
 </instance>
 <instance part="F1" gate="G$1" x="25.4" y="20.32" smashed="yes">
@@
 <wire x1="135.89" y1="66.04" x2="129.54" y2="66.04" width="0.1524" layer="91"/>
 <pinref part="K2" gate="G$1" pin="A"/>
+<wire x1="129.54" y1="66.04" x2="83.82" y2="66.04" width="0.1524" layer="91"/>
+<wire x1="83.82" y1="66.04" x2="78.74" y2="66.04" width="0.1524" layer="91"/>
+<wire x1="78.74" y1="66.04" x2="76.2" y2="66.04" width="0.1524" layer="91"/>
 <wire x1="78.74" y1="38.1" x2="83.82" y2="38.1" width="0.1524" layer="91"/>
 <wire x1="83.82" y1="38.1" x2="129.54" y2="38.1" width="0.1524" layer="91"/>
 <wire x1="129.54" y1="38.1" x2="129.54" y2="66.04" width="0.1524" layer="91"/>
+<pinref part="K1" gate="G$1" pin="A"/>
+<junction x="78.74" y="66.04"/>
+<junction x="129.54" y="66.04"/>
 <label x="137.16" y="66.04" size="1.778" layer="95" xref="yes"/>
-<pinref part="K1" gate="G$1" pin="A"/>
-<wire x1="78.74" y1="66.04" x2="76.2" y2="66.04" width="0.1524" layer="91"/>
-<wire x1="78.74" y1="66.04" x2="83.82" y2="66.04" width="0.1524" layer="91"/>
-<junction x="78.74" y="66.04"/>
-<wire x1="129.54" y1="66.04" x2="83.82" y2="66.04" width="0.1524" layer="91"/>
-<junction x="129.54" y="66.04"/>
+<pinref part="D1" gate="G$1" pin="A"/>
+<junction x="83.82" y="66.04"/>
+<pinref part="D2" gate="G$1" pin="A"/>
+<wire x1="83.82" y1="40.64" x2="83.82" y2="38.1" width="0.1524" layer="91"/>
+<junction x="83.82" y="38.1"/>
 </segment>
 <segment>
@@
 <wire x1="83.82" y1="73.66" x2="78.74" y2="73.66" width="0.1524" layer="91"/>
 <wire x1="78.74" y1="71.12" x2="78.74" y2="73.66" width="0.1524" layer="91"/>
+<pinref part="D1" gate="G$1" pin="C"/>
+<wire x1="83.82" y1="71.12" x2="83.82" y2="73.66" width="0.1524" layer="91"/>
+<junction x="83.82" y="73.66"/>
 </segment>
 </net>
@@
 <net name="N$9" class="0">
 <segment>
-<pinref part="K2" gate="G$1" pin="K"/>
-<wire x1="78.74" y1="43.18" x2="83.82" y2="43.18" width="0.1524" layer="91"/>
 <pinref part="JY3" gate="G$1" pin="C"/>
 <wire x1="88.9" y1="45.72" x2="83.82" y2="45.72" width="0.1524" layer="91"/>
-<wire x1="83.82" y1="45.72" x2="83.82" y2="43.18" width="0.1524" layer="91"/>
+<pinref part="K2" gate="G$1" pin="K"/>
+<wire x1="83.82" y1="45.72" x2="78.74" y2="45.72" width="0.1524" layer="91"/>
+<wire x1="78.74" y1="43.18" x2="78.74" y2="45.72" width="0.1524" layer="91"/>
+<pinref part="D2" gate="G$1" pin="C"/>
+<junction x="83.82" y="45.72"/>
 </segment>
 </net>
@@
 <wire x1="33.02" y1="66.04" x2="43.18" y2="66.04" width="0.1524" layer="91"/>
 <label x="33.02" y="66.04" size="1.778" layer="95" rot="R180" xref="yes"/>
+<pinref part="JP1" gate="G$1" pin="1"/>
 <wire x1="43.18" y1="66.04" x2="58.42" y2="66.04" width="0.1524" layer="91"/>
+<wire x1="27.94" y1="58.42" x2="43.18" y2="58.42" width="0.1524" layer="91"/>
+<wire x1="43.18" y1="58.42" x2="43.18" y2="66.04" width="0.1524" layer="91"/>
+<junction x="43.18" y="66.04"/>
 </segment>
 <segment>
@@
 <wire x1="58.42" y1="38.1" x2="43.18" y2="38.1" width="0.1524" layer="91"/>
 <label x="33.02" y="38.1" size="1.778" layer="95" rot="R180" xref="yes"/>
+<pinref part="JP2" gate="G$1" pin="1"/>
 <wire x1="43.18" y1="38.1" x2="33.02" y2="38.1" width="0.1524" layer="91"/>
-</segment>
-<segment>
+<wire x1="27.94" y1="33.02" x2="43.18" y2="33.02" width="0.1524" layer="91"/>
+<wire x1="43.18" y1="33.02" x2="43.18" y2="38.1" width="0.1524" layer="91"/>
+<junction x="43.18" y="38.1"/>
+</segment>
+<segment>
