File: PCB/PCB_OnOnfre_SINGLE_rev1/PCB_OnOnfre_SINGLE_rev1.sch (EAGLE design)
At the start: 24 parts, among them J1 9PIN 2.54MM, J3Y S8050, J7 8p, U2 esp12

Commit message: rev1.0 single
Parts:
- added U$2: RELAYPTH, SRD-05VDC-SL-C:RELAYPTH
Connections:
- removed net LINE_ONE_OUT: X1-3.KL
- removed net LINE_TWO_OUT: X1-4.KL
- new net LINE_OUT_NC: U$2.SWCLOSE, X1-3.KL
- new net LINE_OUT_NO: U$2.SWOPEN, X1-4.KL
- net LINE_L: now also U$2.SWCOMMON
- net N$1: now also U$2.COIL0
- net VCC: now also U$2.COIL1
Changed lines of the file:
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@@
 <part name="R6" library="resistor" library_urn="urn:adsk.eagle:library:348" deviceset="R-EU_" device="R0603" package3d_urn="urn:adsk.eagle:package:26057/1" value="220k"/>
 <part name="R7" library="resistor" library_urn="urn:adsk.eagle:library:348" deviceset="R-EU_" device="R0603" package3d_urn="urn:adsk.eagle:package:26057/1" value="100k"/>
+<part name="U$2" library="SRD-05VDC-SL-C" deviceset="RELAY" device="PTH"/>
 </parts>
 <sheets>
@@
 <attribute name="NAME" x="224.5614" y="80.01" size="1.778" layer="95" rot="R90"/>
 <attribute name="VALUE" x="229.362" y="80.01" size="1.778" layer="96" rot="R90"/>
+</instance>
+<instance part="U$2" gate="G$1" x="66.04" y="66.04" smashed="yes" rot="R180">
+<attribute name="NAME" x="73.66" y="57.912" size="1.778" layer="95" rot="R180"/>
+<attribute name="VALUE" x="73.66" y="76.2" size="1.778" layer="96" rot="R180"/>
 </instance>
 </instances>
@@
 <pinref part="D1" gate="G$1" pin="A"/>
 <junction x="83.82" y="66.04"/>
+<pinref part="U$2" gate="G$1" pin="COIL1"/>
+<wire x1="76.2" y1="66.04" x2="76.2" y2="60.96" width="0.1524" layer="91"/>
 </segment>
 <segment>
@@
 <pinref part="J3Y" gate="G$1" pin="C"/>
 <wire x1="91.44" y1="73.66" x2="83.82" y2="73.66" width="0.1524" layer="91"/>
-<wire x1="83.82" y1="73.66" x2="78.74" y2="73.66" width="0.1524" layer="91"/>
-<wire x1="78.74" y1="71.12" x2="78.74" y2="73.66" width="0.1524" layer="91"/>
+<wire x1="83.82" y1="73.66" x2="76.2" y2="71.12" width="0.1524" layer="91"/>
 <pinref part="D1" gate="G$1" pin="C"/>
 <wire x1="83.82" y1="71.12" x2="83.82" y2="73.66" width="0.1524" layer="91"/>
 <junction x="83.82" y="73.66"/>
+<pinref part="U$2" gate="G$1" pin="COIL0"/>
 </segment>
 </net>
@@
 <wire x1="17.78" y1="25.4" x2="30.48" y2="25.4" width="0.1524" layer="91"/>
 <label x="30.48" y="25.4" size="1.778" layer="95" xref="yes"/>
-</segment>
-</net>
-<net name="LINE_TWO_OUT" class="1">
-<segment>
-<label x="22.86" y="10.16" size="1.778" layer="95" xref="yes"/>
-<pinref part="X1" gate="-4" pin="KL"/>
-<wire x1="17.78" y1="10.16" x2="22.86" y2="10.16" width="0.1524" layer="91"/>
 </segment>
 </net>
@@
 </segment>
 </net>
-<net name="LINE_ONE_OUT" class="1">
-<segment>
-<wire x1="58.42" y1="71.12" x2="35.56" y2="71.12" width="0.1524" layer="91"/>
-<label x="35.56" y="71.12" size="1.778" layer="95" rot="R180" xref="yes"/>
-</segment>
-<segment>
-<label x="22.86" y="15.24" size="1.778" layer="95" xref="yes"/>
-<pinref part="X1" gate="-3" pin="KL"/>
-<wire x1="17.78" y1="15.24" x2="22.86" y2="15.24" width="0.1524" layer="91"/>
-</segment>
-</net>
 <net name="LINE_L" class="1">
 <segment>
 <label x="33.02" y="66.04" size="1.778" layer="95" rot="R180" xref="yes"/>
 <wire x1="33.02" y1="66.04" x2="58.42" y2="66.04" width="0.1524" layer="91"/>
+<pinref part="U$2" gate="G$1" pin="SWCOMMON"/>
 </segment>
 <segment>
@@
 </segment>
 </net>
+<net name="LINE_OUT_NO" class="1">
+<segment>
+<wire x1="58.42" y1="71.12" x2="35.56" y2="71.12" width="0.1524" layer="91"/>
+<label x="35.56" y="71.12" size="1.778" layer="95" rot="R180" xref="yes"/>
+<pinref part="U$2" gate="G$1" pin="SWOPEN"/>
+</segment>
+<segment>
+<label x="22.86" y="10.16" size="1.778" layer="95" xref="yes"/>
+<pinref part="X1" gate="-4" pin="KL"/>
+<wire x1="17.78" y1="10.16" x2="22.86" y2="10.16" width="0.1524" layer="91"/>
+</segment>
+</net>
+<net name="LINE_OUT_NC" class="0">
+<segment>
+<pinref part="U$2" gate="G$1" pin="SWCLOSE"/>
+<wire x1="58.42" y1="60.96" x2="20.32" y2="60.96" width="0.1524" layer="91"/>
+<label x="20.32" y="60.96" size="1.778" layer="95" rot="R180" xref="yes"/>
+</segment>
+<segment>
+<label x="22.86" y="15.24" size="1.778" layer="95" xref="yes"/>
+<pinref part="X1" gate="-3" pin="KL"/>
+<wire x1="17.78" y1="15.24" x2="22.86" y2="15.24" width="0.1524" layer="91"/>
+</segment>
+</net>
