File: PCB/PCB_OnOnfre_SINGLE_rev1/PCB_OnOnfre_SINGLE_rev1.brd (EAGLE design)
At the start: 44 x 41.7 mm, 32 parts, among them J1 9PIN 2.54MM, J3Y S8050, J7 8p, K1 OMRON-G3MB-202P-SSR2, K2 OMRON-G3MB-202P-SSR2, U2 esp12

Commit message: s
Parts:
- removed D2: 1N4148, diode:SOD80C
- removed JP1, JP2: (no value), pinhead:1X01
- removed JY3: S8050, semicon-smd-ipc:SOT23
- removed K1, K2: OMRON-G3MB-202P-SSR2, Omron G3MB 202p SSR:OMRON-G3MB-202P-SSR
- removed R1, R2: 10k, resistor:R0603
- moved D1 35.2 mm to (7.36, 24.0)
Connections:
- removed net N$13: JY3.1, R1.2, R2.2
- removed net N$9: D2.C, JY3.3, K2.4
- net GND: no longer JY3.2, R2.1
- net GPIO05: no longer R1.1
- net LINE_L: no longer JP1.1, JP2.1, K1.1, K2.1
- net LINE_ONE_OUT: no longer K1.2
- net LINE_TWO_OUT: no longer K2.2
- net N$1: no longer K1.4
- net VCC: no longer D2.A, K1.3, K2.3
Routing:
- net N$1: track 30.4 -> 2.30 mm
- net LINE_L: track 37.9 -> 10.4 mm
- net N$9: track 20.6 -> 0.00 mm
- net LINE_TWO_OUT: track 13.5 -> 0.00 mm
- net GPIO05: track 16.3 -> 3.85 mm
- net VCC: track 67.7 -> 58.7 mm
- net LINE_ONE_OUT: track 7.16 -> 0.00 mm
- net N$13: track 4.10 -> 0.00 mm
- net GND: track 88.6 -> 86.3 mm
- removed copper zone on layer 1, net GND
- removed copper zone on layer 16, net GND
Other:
- outline, holes or cut-outs redrawn

Commit message: rev1.0 single
Parts:
- added U$2: RELAYPTH, SRD-05VDC-SL-C:SRD-05VDC-SL-C
- moved D1 10.6 mm to (17.6, 26.3), turned to 90 degrees
- moved X1 1.32 mm to (24.5, 5.29)
Connections:
- removed net LINE_ONE_OUT: X1.3
- removed net LINE_TWO_OUT: X1.4
- new net LINE_OUT_NC: U$2.SWCLOSED, X1.3
- new net LINE_OUT_NO: U$2.SWOPEN, X1.4
- net LINE_L: now also U$2.SWCOMMON
- net N$1: now also U$2.COIL0
- net VCC: now also U$2.COIL1
Routing:
- net N$1: track 2.30 -> 30.1 mm
- net LINE_OUT_NC: track 0.00 -> 17.6 mm
- net GPIO0: track 41.2 -> 56.0 mm, vias 1 -> 0
- net VCC: track 58.7 -> 70.2 mm, vias 0 -> 2
- net LINE_OUT_NO: track 0.00 -> 6.03 mm
- net LINE_L: track 10.4 -> 16.3 mm
- net GND: track 86.3 -> 84.3 mm
- net N$2: track 7.00 -> 8.31 mm
- net NEUTRAL_IN: track 19.1 -> 18.4 mm
Other:
- board size 44 x 41.7 mm -> 44 x 42.3 mm
- board text added: "rev1.0"
- board text removed: "N"
- board text removed: "rev5.0"

Commit message: pcb single
Parts:
- removed U$2: RELAYPTH, SRD-05VDC-SL-C:SRD-05VDC-SL-C
- added RLY1: SRD-05VDC-SL-C, Spark:SRD-5VDC-SL-C
- moved X1 3.80 mm to (24.6, 1.49)
Connections:
- net LINE_L: now also RLY1.COMMON; no longer U$2.SWCOMMON
- net LINE_OUT_NC: now also RLY1.CLOSED, X1.4; no longer U$2.SWCLOSED, X1.3
- net LINE_OUT_NO: now also RLY1.OPEN, X1.3; no longer U$2.SWOPEN, X1.4
- net N$1: now also RLY1.COIL2; no longer U$2.COIL0
- net VCC: now also RLY1.COIL1; no longer U$2.COIL1
Routing:
- net LINE_L: track 16.3 -> 33.8 mm
- net N$1: track 30.1 -> 38.4 mm
- net VCC: track 70.2 -> 76.4 mm, vias 2 -> 0
- net N$2: track 8.31 -> 12.2 mm
- net LINE_OUT_NC: track 17.6 -> 21.0 mm
- net GPIO0: track 56.0 -> 52.7 mm
- net LINE_OUT_NO: track 6.03 -> 7.79 mm
- net NEUTRAL_IN: track 18.4 -> 20.1 mm
Other:
- board size 44 x 42.3 mm -> 44 x 46.8 mm
