File: PCB/PCB_OnOnfre_DUAL_rev5.1/OnOnfre_DevBoard.brd (EAGLE design)
At the start: 44 x 41.7 mm, 32 parts, among them J1 9PIN 2.54MM, J3Y S8050, J7 8p, K1 OMRON-G3MB-202P-SSR2, K2 OMRON-G3MB-202P-SSR2, U2 esp12

Commit message: rev5.1
remoção de diodos e slot para relés mecanicos
Parts:
- removed D1, D2: 1N4148, diode:SOD80C
- removed JP1, JP2: (no value), pinhead:1X01
- moved FLASH 0.21 mm to (36.5, 31.0)
- moved RESET 0.21 mm to (36.5, 38.6)
Connections:
- net LINE_L: no longer JP1.1, JP2.1
- net N$1: no longer D1.C
- net N$9: no longer D2.C
- net VCC: no longer D1.A, D2.A
Routing:
- net LINE_L: track 37.9 -> 21.1 mm
- net GND: track 88.6 -> 84.6 mm
- net N$9: track 20.6 -> 18.2 mm
- net N$1: track 30.4 -> 28.2 mm
Other:
- board text added: "rev5.1"
- board text removed: "rev5.0"
