File: PCB/PCB_OnOnfre_DUAL_rev5.1/OnOnfre_DevBoard.sch (EAGLE design)
At the start: 30 parts, among them J1 9PIN 2.54MM, J3Y S8050, J7 8p, K1 PA1A-6VV, K2 PA1A-6VV, U2 esp12

Commit message: board
Parts:
- removed D1, D2: 1N4148, diode:DIODE-SOD80C
- K1, K2: value PA1A-6VV -> OMRON-G3MB-202P-SSR2; device relay:PA1A-6VV -> Omron G3MB 202p SSR:OMRON-G3MB-202P-SSR2
Connections:
- net LINE_L: now also K1.DS1, K2.DS1; no longer K12.P, K22.P
- net LINE_ONE_OUT: now also K1.DS2; no longer K12.S
- net LINE_TWO_OUT: now also K2.DS2; no longer K22.S
- net N$1: now also K1.K; no longer D1.A, K11.2
- net N$9: now also K2.K; no longer D2.A, K21.2
- net VCC: now also K1.A, K2.A; no longer D1.C, D2.C, K11.1, K21.1
