File: PCB/PCB_OnOnfre_DUAL_BETA Solenoid/OnOnfre_DevBoard.brd (EAGLE design)
At the start: 44.1 x 43.8 mm, 29 parts, among them J1 9PIN 2.54MM, J3Y S8050, J7 8p, K1 G5Q-1-DC12, K2 G5Q-1-DC12, U2 esp12

Commit message: s
Parts:
- added C5: (no value), rcl:C102-043X133
- added R5: (no value), resistor:R2512
- moved F1 3.83 mm to (15.6, 18.4)
- moved X1 1.98 mm to (10.9, 5.05)
- moved K2 0.61 mm to (28.9, 13.1)
- moved K1 0.29 mm to (39.4, 13.1)
Connections:
- new net N$3: K1.2, R5.2
- new net N$4: C5.2, R5.1
- net LINE_DOWN_OUT: now also K2.4; no longer K2.3
- net LINE_IN_FUSED: now also K1.3; no longer K1.4, K2.4
- net LINE_UP_OUT: now also K2.3; no longer K1.3
- net N$2: now also C5.1; no longer K1.2
Routing:
- net N$4: track 0.00 -> 20.9 mm
- net LINE_IN_FUSED: track 21.9 -> 35.9 mm, vias 0 -> 1
- net LINE_UP_OUT: track 37.7 -> 26.4 mm
- net LINE_DOWN_OUT: track 16.4 -> 8.21 mm
- net N$2: track 10.7 -> 15.3 mm
- net N$3: track 0.00 -> 3.93 mm
- net VCC: track 88.0 -> 89.7 mm
- net LINE_L: track 12.7 -> 14.2 mm
- net NEUTRAL_IN: track 8.82 -> 10.2 mm
- net N$9: track 34.2 -> 33.6 mm
Other:
- outline, holes or cut-outs redrawn

Commit message: snub
Connections:
- removed net N$2: C5.1, K2.2
- net LINE_IN_FUSED: now also C5.1
- net N$3: now also K2.2
Routing:
- net N$2: track 15.3 -> 0.00 mm
- net LINE_IN_FUSED: track 35.9 -> 46.2 mm
Changed lines of the file:
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@@
 <?xml version="1.0" encoding="utf-8"?>
 <!DOCTYPE eagle SYSTEM "eagle.dtd">
-<eagle version="9.2.2">
+<eagle version="9.1.3">
 <drawing>
 <settings>
-<setting alwaysvectorfont="yes"/>
+<setting alwaysvectorfont="no"/>
 <setting verticaltext="up"/>
 </settings>
@@
 <wire x1="18.427865625" y1="14.86178125" x2="18.25105625" y2="15.038590625" width="1.27" layer="1"/>
 <wire x1="18.25105625" y1="15.038590625" x2="18.25105625" y2="18.42916875" width="1.27" layer="1"/>
-</signal>
-<signal name="N$2">
-<contactref element="K2" pad="2"/>
 <contactref element="C5" pad="1"/>
-<wire x1="32.8709" y1="11.93035625" x2="29.359759375" y2="15.441496875" width="1.27" layer="1"/>
 <wire x1="29.359759375" y1="15.441496875" x2="23.06115625" y2="15.441496875" width="1.27" layer="1"/>
 <wire x1="23.06115625" y1="15.441496875" x2="22.20686875" y2="16.295784375" width="1.27" layer="1"/>
 <wire x1="22.20686875" y1="16.295784375" x2="22.20686875" y2="19.104521875" width="1.27" layer="1"/>
+<wire x1="23.613959375" y1="15.707515625" x2="23.06115625" y2="15.441496875" width="0" layer="19" extent="1-16"/>
 </signal>
 <signal name="N$3">
@@
 <wire x1="43.40171875" y1="11.9303875" x2="41.905053125" y2="13.427053125" width="1.27" layer="1"/>
 <wire x1="41.905053125" y1="13.427053125" x2="41.905053125" y2="15.240303125" width="1.27" layer="1"/>
+<contactref element="K2" pad="2"/>
+<wire x1="32.8709" y1="11.93035625" x2="41.905053125" y2="13.427053125" width="0" layer="19" extent="1-1"/>
 </signal>
 <signal name="N$4">

Commit message: estores
Parts:
- removed C5: (no value), rcl:C102-043X133
- removed R5: (no value), resistor:R2512
- added C6: (no value), rcl:C102-043X133
- added R12: (no value), resistor:R2512
- added R13: VARISTORS07K230, varistor:S07K230
- moved X1 2.84 mm to (13.7, 4.46)
- moved F1 0.58 mm to (15.1, 18.4)
Connections:
- removed net N$4: C5.2, R5.1
- new net N$5: C6.2, R12.1
- net LINE_IN_FUSED: now also R13.1; no longer C5.1
- net N$3: now also R12.2; no longer R5.2
- net NEUTRAL_IN: now also C6.1, R13.2
Routing:
- net N$4: track 20.9 -> 0.00 mm
- net NEUTRAL_IN: track 10.2 -> 30.4 mm
- net N$5: track 0.00 -> 16.1 mm
- net LINE_IN_FUSED: track 46.2 -> 34.3 mm, vias 1 -> 0
- net N$3: track 3.93 -> 15.0 mm
- net LINE_UP_OUT: track 26.4 -> 21.8 mm
- net LINE_DOWN_OUT: track 8.21 -> 4.55 mm
- added copper zone on layer 1, net GND
- added copper zone on layer 16, net GND
Other:
- outline, holes or cut-outs redrawn
