File: PCB/PCB_OnOnfre_DUAL_BETA Solenoid/OnOnfre_DevBoard.sch (EAGLE design)
At the start: 25 parts, among them J3Y S8050, J7 8p, U2 esp12

Commit message: 10A
Parts:
- removed D3: 1N4004, Seeed-Diode:DIODE-GEN-PURPOSE-1KV-1A(DO-214AC)
- removed U$2: HKLPM01, HKLPM01:HKLPM01
- removed U$3: HF46F, HF46F:HF46F
- added C1, C2: 22uF, Seeed-Capacitor:CERAMIC-1NF-1KV-10%-X7R(1206)
- added C3: 100uF, Seeed-Capacitor:CERAMIC-1NF-1KV-10%-X7R(1206)
- added K1, K2: G5Q-1-DC12, G5Q-1-DC12:G5Q-1-DC12
- added R6: 220k, resistor:R-EU_R0603
- added R7: 100k, resistor:R-EU_R0603
- C4: value 100NF -> 100uF
- D1, D2: value 1N4007 -> 1N4148; device Seeed-Diode:DIODE-GEN-PURPOSE-1KV-1A(DO-214AC) -> diode:DIODE-SOD80C
- F1: value FUSE -> 1812L010; device SparkFun-Fuses:PPTC_PTH -> polyfuse-smd_10:1812L010
- J1: value (none) -> 9PIN 2.54MM
- U$1: value HF46F -> HLK-PM01; device HF46F:HF46F -> HLK-PM01:HLK-PM01
Connections:
- removed net 5V: D1.-, D2.-, D3.-, J1.9, U$1.C1, U$3.C1
- removed net LINE_IN: U$2.AC2, X1-1.KL
- removed net NEUTRAL_IN_FUSED: F1.2, U$1.L1, U$3.L1
- removed net NEUTRAL_ONE_OUT: U$1.L2, X1-3.KL
- removed net NEUTRAL_TWO_OUT: U$3.L2, X1-4.KL
- new net A0: J7.7, R6.2
- new net COM: K1.2, K2.2
- new net LINE_DOWN_OUT: K2.3, X1-4.KL
- new net LINE_FUSED: F1.1, K1.4, K2.4
- new net LINE_L: F1.2, U$1.AC1, X1-2.KL
- new net LINE_UP_OUT: K1.3, X1-3.KL
- net 3V3: now also C1.1
- net ADC: now also R6.1, R7.2; no longer J7.7
- net GND: now also C1.2, C2.2, C3.2, R7.1, U$1.DC-; no longer U$2.-VO
- net N$1: now also D1.A, K1.5; no longer D1.+, U$1.C2
- net N$9: now also D2.A, K2.5; no longer D2.+, U$3.C2
- net NEUTRAL_IN: now also U$1.AC2, X1-1.KL; no longer F1.1, U$2.AC1, X1-2.KL
- net VCC: now also C2.1, C3.1, D1.C, D2.C, J1.9, K1.1, K2.1, U$1.DC+; no longer D3.+, U$2.+VO
Other:
- note removed: "BH ON OFRE 12"
- note removed: "ESP8266-12"
- moved on the sheet: C4, J3Y, JY3, R1, R2, R3, R4, X1-1, X1-2, X1-3, X1-4
