File: PCB/PCB_OnOnfre_SINGLE_BETA1 Solenoid/PCB_OnOnfre_SINGLE_BETA1 Solenoid.sch (EAGLE design)
At the start: 32 parts, among them J1 9PIN 2.54MM, J3Y S8050, J7 8p, K1 G5Q-1-DC12, K2 G5Q-1-DC12, U2 esp12

Commit message: bl
Parts:
- removed D2: 1N4148, diode:DIODE-SOD80C
- removed JY3: S8050, semicon-smd-ipc:NPN-TRANSISTOR_SOT23
- removed K1: G5Q-1-DC12, G5Q-1-DC12:G5Q-1-DC12
- removed R1, R2: 10k, resistor:R-EU_R0603
- removed X1: (no value), con-wago-500:W237-4
- added X2: (no value), con-wago-500:W237-103
- C1, C2: value 1NF -> 22uF
- C3, C4: value 1NF -> 100uF
- K2: value G5Q-1-DC12 -> E3206S; device G5Q-1-DC12:G5Q-1-DC12 -> relay:E3206S
Connections:
- removed net LINE_DOWN_OUT: K2.4, X1-4.KL
- removed net LINE_UP_OUT: K2.3, X1-3.KL
- removed net N$13: JY3.B, R1.2, R2.2
- removed net N$3: K1.2, K2.2, R12.2
- removed net N$9: D2.A, JY3.C, K2.5
- new net LINE_OUT: C6.1, K22.S, X2-3.KL
- net GND: no longer JY3.E, R2.1
- net GPIO05: no longer R1.1
- net LINE_IN_FUSED: now also K22.P, R12.2; no longer C6.1, K1.3
- net LINE_L: now also X2-2.KL; no longer X1-2.KL
- net N$1: now also K21.1; no longer K1.5
- net NEUTRAL_IN: now also X2-1.KL; no longer X1-1.KL
- net VCC: now also K21.2; no longer D2.C, K1.1, K2.1
