File: PCB/PCB_OnOnfre_DUAL_BETA1 Solenoid/OnOnfre_DevBoard.sch (EAGLE design)
At the start: 32 parts, among them J1 9PIN 2.54MM, J3Y S8050, J7 8p, K1 G5Q-1-DC12, K2 G5Q-1-DC12, U2 esp12

Commit message: estores rev1
Parts:
- removed C2, C3: 1NF, Seeed-Capacitor:CERAMIC-1NF-1KV-10%-X7R(1206)
Connections:
- net GND: no longer C2.2, C3.2
- net VCC: no longer C2.1, C3.1
Changed lines of the file:
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@@
 <part name="X1" library="con-wago-500" library_urn="urn:adsk.eagle:library:195" deviceset="W237-4" device="" package3d_urn="urn:adsk.eagle:package:10695/1"/>
 <part name="C1" library="Seeed-Capacitor" library_urn="urn:adsk.eagle:library:464" deviceset="CERAMIC-1NF-1KV-10%-X7R?(1206)" device="" package3d_urn="urn:adsk.eagle:package:32384/1" value="1NF"/>
-<part name="C2" library="Seeed-Capacitor" library_urn="urn:adsk.eagle:library:464" deviceset="CERAMIC-1NF-1KV-10%-X7R?(1206)" device="" package3d_urn="urn:adsk.eagle:package:32384/1" value="1NF"/>
-<part name="C3" library="Seeed-Capacitor" library_urn="urn:adsk.eagle:library:464" deviceset="CERAMIC-1NF-1KV-10%-X7R?(1206)" device="" package3d_urn="urn:adsk.eagle:package:32384/1" value="1NF"/>
 <part name="U$1" library="HLK-PM01" deviceset="HLK-PM01" device=""/>
 <part name="F1" library="polyfuse-smd_10" deviceset="?" device="1812L" technology="010"/>
@@
 <attribute name="VALUE" x="185.42" y="110.49" size="1.27" layer="96" ratio="10" rot="R270"/>
 </instance>
-<instance part="C2" gate="G$1" x="149.86" y="106.68" smashed="yes" rot="R270">
-<attribute name="NAME" x="151.13" y="110.49" size="1.27" layer="95" ratio="10" rot="R270"/>
-<attribute name="VALUE" x="147.32" y="110.49" size="1.27" layer="96" ratio="10" rot="R270"/>
-</instance>
-<instance part="C3" gate="G$1" x="157.48" y="106.68" smashed="yes" rot="R270">
-<attribute name="NAME" x="158.75" y="110.49" size="1.27" layer="95" ratio="10" rot="R270"/>
-<attribute name="VALUE" x="154.94" y="110.49" size="1.27" layer="96" ratio="10" rot="R270"/>
-</instance>
 <instance part="U$1" gate="G$1" x="223.52" y="144.78" smashed="yes">
 <attribute name="NAME" x="213.36" y="137.16" size="1.778" layer="94"/>
@@
 <label x="167.64" y="99.06" size="1.778" layer="95" rot="R270" xref="yes"/>
 <wire x1="167.64" y1="101.6" x2="167.64" y2="99.06" width="0.1524" layer="91"/>
-<wire x1="149.86" y1="101.6" x2="157.48" y2="101.6" width="0.1524" layer="91"/>
-<wire x1="157.48" y1="101.6" x2="167.64" y2="101.6" width="0.1524" layer="91"/>
-<wire x1="149.86" y1="102.87" x2="149.86" y2="101.6" width="0.1524" layer="91"/>
-<pinref part="C2" gate="G$1" pin="2"/>
-<pinref part="C3" gate="G$1" pin="2"/>
-<wire x1="157.48" y1="102.87" x2="157.48" y2="101.6" width="0.1524" layer="91"/>
 <wire x1="167.64" y1="101.6" x2="182.88" y2="101.6" width="0.1524" layer="91"/>
 <wire x1="182.88" y1="101.6" x2="187.96" y2="101.6" width="0.1524" layer="91"/>
@@
 <junction x="182.88" y="101.6"/>
 <junction x="167.64" y="101.6"/>
-<junction x="157.48" y="101.6"/>
 </segment>
 <segment>
@@
 <segment>
 <pinref part="AMS1117" gate="G$1" pin="IN"/>
-<wire x1="160.02" y1="111.76" x2="157.48" y2="111.76" width="0.1524" layer="91"/>
 <label x="147.32" y="111.76" size="1.778" layer="95" rot="R180" xref="yes"/>
-<wire x1="157.48" y1="111.76" x2="149.86" y2="111.76" width="0.1524" layer="91"/>
-<wire x1="149.86" y1="111.76" x2="147.32" y2="111.76" width="0.1524" layer="91"/>
-<wire x1="149.86" y1="111.76" x2="149.86" y2="110.49" width="0.1524" layer="91"/>
-<wire x1="157.48" y1="111.76" x2="157.48" y2="110.49" width="0.1524" layer="91"/>
-<pinref part="C2" gate="G$1" pin="1"/>
-<pinref part="C3" gate="G$1" pin="1"/>
-<junction x="149.86" y="111.76"/>
-<junction x="157.48" y="111.76"/>
-</segment>
-<segment>
+<wire x1="160.02" y1="111.76" x2="147.32" y2="111.76" width="0.1524" layer="91"/>
+</segment>
+<segment>
