File: PCB/ONOFRE_WIRE_SHIELD/ONOFRE_WIRE_SHIELD.sch (EAGLE design)
At the start: 9 parts, among them J1 9PIN 2.54MM, J7 8p

Commit message: shield v2
Parts:
- added J3, J4, J6: (no value), SparkFun-Connectors:CONN_02
- added J5: (no value), SparkFun-Connectors:CONN_03
- added R6: 220k, resistor:R-EU_R0603
- added R7: 100k, resistor:R-EU_R0603
Connections:
- new net ADC: J6.1, R6.1, R7.2
- net 3V3: now also J3.1, J5.3
- net A0: now also R6.2
- net GND: now also J4.1, J5.2, J6.2, R7.1
- net GPIO14: now also J4.2
- net GPIO16: now also J3.2
- net VCC: now also J5.1
Other:
- moved on the sheet: 3V3, J7, RST
