File: PCB/ONOFRE_ESTORES_COVERS_R1.1/ONOFRE_ESTORES_COVERS_R1.1.sch (EAGLE design)
At the start: 30 parts, among them J1 9PIN 2.54MM, J3Y S8050, J7 8p, K1 G5Q-1-DC12, K2 G5Q-1-DC12, U2 esp12

Commit message: estores
Parts:
- C6: value (none) -> 47nf 400V
- R12: value 100R -> 100R 1w
Changed lines of the file:
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@@
 <part name="K1" library="G5Q-1-DC12" deviceset="G5Q-1-DC12" device=""/>
 <part name="K2" library="G5Q-1-DC12" deviceset="G5Q-1-DC12" device=""/>
-<part name="R12" library="resistor" library_urn="urn:adsk.eagle:library:348" deviceset="R-EU_" device="R2512" package3d_urn="urn:adsk.eagle:package:23545/2" value="100R"/>
-<part name="C6" library="rcl" library_urn="urn:adsk.eagle:library:334" deviceset="C-EU" device="102-043X133" package3d_urn="urn:adsk.eagle:package:23647/1"/>
+<part name="R12" library="resistor" library_urn="urn:adsk.eagle:library:348" deviceset="R-EU_" device="R2512" package3d_urn="urn:adsk.eagle:package:23545/2" value="100R 1w"/>
+<part name="C6" library="rcl" library_urn="urn:adsk.eagle:library:334" deviceset="C-EU" device="102-043X133" package3d_urn="urn:adsk.eagle:package:23647/1" value="47nf 400V"/>
 <part name="R5" library="varistor" library_urn="urn:adsk.eagle:library:410" deviceset="VARISTOR" device="S07K230" package3d_urn="urn:adsk.eagle:package:30547/1"/>
 </parts>
